File: KiCad/TinyTiM.kicad_pcb (KiCad board)
At the start: 2 copper layers, 243.8 x 121.9 mm, 129 parts, among them P101 PWR_NW, P102 DO_N1, P103 DO_N2, P104 DI_N1, P105 DI_N2, P106 PWR_NE, P107 PWR_W, P108 PWR_E, P109 DI_W2, P110 DO_E2, P111 DI_W1, P112 DO_E1, P113 PWR_SW, P114 DI_S1, P115 DI_S2, P116 DO_S1, P117 DO_S2, P118 PWR_SE, P119 DO_H_SER, P120 DI_A_SER, P121 DI_A_SER, P122 DO_H_SER, P123 DI_A_Ser, P124 DO_H_Ser, P125 G>H, P126 F>G, P127 E>F, P128 D>E, P129 C>D, P130 B>C, P131 A>B, U101 RGB_WS2811, U102 RGB_WS2811, U103 RGB_WS2811, U104 RGB_WS2811, U105 RGB_WS2811, U106 RGB_WS2811, U107 RGB_WS2811, U108 RGB_WS2811, U201 RGB_WS2811, U202 RGB_WS2811, U203 RGB_WS2811, U204 RGB_WS2811, U205 RGB_WS2811, U206 RGB_WS2811, U207 RGB_WS2811, U208 RGB_WS2811, U301 RGB_WS2811, U302 RGB_WS2811, U303 RGB_WS2811, U304 RGB_WS2811, U305 RGB_WS2811, U306 RGB_WS2811, U307 RGB_WS2811, U308 RGB_WS2811, U401 RGB_WS2811, U402 RGB_WS2811, U403 RGB_WS2811, U404 RGB_WS2811, U405 RGB_WS2811, U406 RGB_WS2811, U407 RGB_WS2811, U408 RGB_WS2811, U501 RGB_WS2811, U502 RGB_WS2811, U503 RGB_WS2811, U504 RGB_WS2811, U505 RGB_WS2811, U506 RGB_WS2811, U507 RGB_WS2811, U508 RGB_WS2811, U601 RGB_WS2811, U602 RGB_WS2811, U603 RGB_WS2811, U604 RGB_WS2811, U605 RGB_WS2811, U606 RGB_WS2811, U607 RGB_WS2811, U608 RGB_WS2811, U701 RGB_WS2811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

Commit message: TinyTiM KiCad work in progress
Routing:
- net GND: track 3075.6 -> 2044.4 mm
- net 5V: track 2759.4 -> 2066.9 mm
- net /Row_H/DO_H: track 730.0 -> 669.6 mm, vias 2 -> 1
- net /Row_A/DO_A: track 462.5 -> 405.8 mm, vias 1 -> 0
- net /Row_G/DO_G: track 396.1 -> 347.9 mm, vias 1 -> 0
- net /Row_B/DO_B: track 444.4 -> 401.4 mm, vias 1 -> 0
- net /Row_D/D_16: track 39.1 -> 0.00 mm, vias 2 -> 0
- net /Row_F/DO_F: track 383.6 -> 348.5 mm, vias 1 -> 0
- net /Row_C/DO_C: track 427.2 -> 396.9 mm, vias 1 -> 0
- net /Row_E/DO_E: track 371.0 -> 349.3 mm, vias 1 -> 0
- net /Row_A/A_12: track 19.0 -> 0.00 mm
- net /Row_H/H_14: track 19.0 -> 0.00 mm
- net /Row_A/A_10: track 18.7 -> 0.00 mm
- net /Row_H/H_10: track 18.5 -> 0.00 mm
- net /Row_H/H_12: track 18.4 -> 0.00 mm
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