File: KiCad/Row_A.sch (KiCad schematic (older format))
At the start: 14 parts, among them U101 RGB_WS2811, U102 RGB_WS2811, U103 RGB_WS2811, U104 RGB_WS2811, U105 RGB_WS2811, U106 RGB_WS2811, U107 RGB_WS2811, U108 RGB_WS2811

Commit message: TinyTiM KiCad work in progress
Parts:
- C101: footprint c_0805 -> TinyTiM_Lib:c_0805
- C117: footprint c_2917 -> TinyTiM_Lib:c_2917
- S101, S102, S103, S104: footprint Screw -> TinyTiM_Lib:Screw
- U101, U102, U103, U104, U105, U106, U107, U108: footprint RGB_WS2811 -> TinyTiM_Lib:RGB_WS2811
Changed lines of the file:
@@
 F 0 "U101" V 1300 1575 60  0000 C CNN
 F 1 "RGB_WS2811" V 1925 1550 60  0000 C CNN
-F 2 "RGB_WS2811" H 1425 1975 60  0001 C CNN
+F 2 "TinyTiM_Lib:RGB_WS2811" H 1425 1975 60  0001 C CNN
 F 3 "" H 1525 1575 60  0001 C CNN
 	1    1525 1575
@@
 F 0 "C101" H 1825 2700 50  0000 L CNN
 F 1 "100n" H 1825 2500 50  0000 L CNN
-F 2 "c_0805" H 1800 2600 50  0001 C CNN
+F 2 "TinyTiM_Lib:c_0805" H 1800 2600 50  0001 C CNN
 F 3 "" H 1800 2600 60  0001 C CNN
 F 4 "CAP CER 0.1UF 25V 10% X7R 0805" H 1800 2800 60  0001 L CNN "Field4"
@@
 F 0 "U102" V 2450 1575 60  0000 C CNN
 F 1 "RGB_WS2811" V 3075 1550 60  0000 C CNN
-F 2 "RGB_WS2811" H 2575 1975 60  0001 C CNN
+F 2 "TinyTiM_Lib:RGB_WS2811" H 2575 1975 60  0001 C CNN
 F 3 "" H 2675 1575 60  0001 C CNN
 	1    2675 1575
@@
 F 0 "U103" V 3600 1575 60  0000 C CNN
 F 1 "RGB_WS2811" V 4225 1550 60  0000 C CNN
-F 2 "RGB_WS2811" H 3725 1975 60  0001 C CNN
+F 2 "TinyTiM_Lib:RGB_WS2811" H 3725 1975 60  0001 C CNN
 F 3 "" H 3825 1575 60  0001 C CNN
 	1    3825 1575
@@
 F 0 "U104" V 4750 1550 60  0000 C CNN
 F 1 "RGB_WS2811" V 5375 1550 60  0000 C CNN
-F 2 "RGB_WS2811" H 4875 1975 60  0001 C CNN
+F 2 "TinyTiM_Lib:RGB_WS2811" H 4875 1975 60  0001 C CNN
 F 3 "" H 4975 1575 60  0001 C CNN
 	1    4975 1575
@@
 F 0 "U105" V 5900 1550 60  0000 C CNN
 F 1 "RGB_WS2811" V 6525 1525 60  0000 C CNN
-F 2 "RGB_WS2811" H 6025 1975 60  0001 C CNN
+F 2 "TinyTiM_Lib:RGB_WS2811" H 6025 1975 60  0001 C CNN
 F 3 "" H 6125 1575 60  0001 C CNN
 	1    6125 1575
@@
 F 0 "U106" V 7050 1550 60  0000 C CNN
 F 1 "RGB_WS2811" V 7675 1550 60  0000 C CNN
-F 2 "RGB_WS2811" H 7175 1975 60  0001 C CNN
+F 2 "TinyTiM_Lib:RGB_WS2811" H 7175 1975 60  0001 C CNN
 F 3 "" H 7275 1575 60  0001 C CNN
 	1    7275 1575
@@
 F 0 "U107" V 8200 1550 60  0000 C CNN
 F 1 "RGB_WS2811" V 8825 1550 60  0000 C CNN
-F 2 "RGB_WS2811" H 8325 1975 60  0001 C CNN
+F 2 "TinyTiM_Lib:RGB_WS2811" H 8325 1975 60  0001 C CNN
 F 3 "" H 8425 1575 60  0001 C CNN
 	1    8425 1575
@@
 F 0 "U108" V 9350 1550 60  0000 C CNN
 F 1 "RGB_WS2811" V 9975 1550 60  0000 C CNN
-F 2 "RGB_WS2811" H 9475 1975 60  0001 C CNN
+F 2 "TinyTiM_Lib:RGB_WS2811" H 9475 1975 60  0001 C CNN
 F 3 "" H 9575 1575 60  0001 C CNN
 	1    9575 1575
@@
 F 0 "S101" V 5380 6650 40  0000 L CNN
 F 1 "CONN_1" H 5300 6705 30  0001 C CNN
-F 2 "Screw" H 5300 6805 30  0001 C CNN
+F 2 "TinyTiM_Lib:Screw" H 5300 6805 30  0001 C CNN
 F 3 "" H 5300 6650 60  0001 C CNN
 	1    5300 6650
@@
 F 0 "S102" V 5580 6650 40  0000 L CNN
 F 1 "CONN_1" H 5500 6705 30  0001 C CNN
-F 2 "Screw" H 5500 6805 30  0001 C CNN
+F 2 "TinyTiM_Lib:Screw" H 5500 6805 30  0001 C CNN
 F 3 "" H 5500 6650 60  0001 C CNN
 	1    5500 6650
@@
 F 0 "S103" V 5780 6650 40  0000 L CNN
 F 1 "CONN_1" H 5700 6705 30  0001 C CNN
-F 2 "Screw" H 5700 6805 30  0001 C CNN
+F 2 "TinyTiM_Lib:Screw" H 5700 6805 30  0001 C CNN
 F 3 "" H 5700 6650 60  0001 C CNN
 	1    5700 6650
@@
 F 0 "S104" V 5980 6650 40  0000 L CNN
 F 1 "CONN_1" H 5900 6705 30  0001 C CNN
-F 2 "Screw" H 5900 6805 30  0001 C CNN
+F 2 "TinyTiM_Lib:Screw" H 5900 6805 30  0001 C CNN
 F 3 "" H 5900 6650 60  0001 C CNN
 	1    5900 6650
@@
 F 0 "C117" H 1375 6725 50  0000 L CNN
 F 1 "47u,8V" H 1375 6625 50  0000 L CNN
-F 2 "c_2917" H 1250 6700 50  0001 C CNN
+F 2 "TinyTiM_Lib:c_2917" H 1250 6700 50  0001 C CNN
 F 3 "" H 1250 6750 60  0001 C CNN
 F 4 "CAP ALUM 47UF 8V 20% SMD" H 1250 6950 60  0001 L CNN "Field4"
