File: KiCad/Row_B.sch (KiCad schematic (older format))
At the start: 10 parts, among them U201 RGB_WS2811, U202 RGB_WS2811, U203 RGB_WS2811, U204 RGB_WS2811, U205 RGB_WS2811, U206 RGB_WS2811, U207 RGB_WS2811, U208 RGB_WS2811

Commit message: TinyTiM KiCad work in progress
Parts:
- C201: footprint c_0805 -> TinyTiM_Lib:c_0805
- C217: footprint c_2917 -> TinyTiM_Lib:c_2917
- U201, U202, U203, U204, U205, U206, U207, U208: footprint RGB_WS2811 -> TinyTiM_Lib:RGB_WS2811
Changed lines of the file:
@@
 F 0 "U201" V 1300 1575 60  0000 C CNN
 F 1 "RGB_WS2811" V 1925 1550 60  0000 C CNN
-F 2 "RGB_WS2811" H 1425 1975 60  0001 C CNN
+F 2 "TinyTiM_Lib:RGB_WS2811" H 1425 1975 60  0001 C CNN
 F 3 "" H 1525 1575 60  0001 C CNN
 	1    1525 1575
@@
 F 0 "C201" H 1825 2700 50  0000 L CNN
 F 1 "100n" H 1825 2500 50  0000 L CNN
-F 2 "c_0805" H 1800 2600 50  0001 C CNN
+F 2 "TinyTiM_Lib:c_0805" H 1800 2600 50  0001 C CNN
 F 3 "" H 1800 2600 60  0001 C CNN
 F 4 "CAP CER 0.1UF 25V 10% X7R 0805" H 1800 2800 60  0001 L CNN "Field4"
@@
 F 0 "U202" V 2450 1575 60  0000 C CNN
 F 1 "RGB_WS2811" V 3075 1550 60  0000 C CNN
-F 2 "RGB_WS2811" H 2575 1975 60  0001 C CNN
+F 2 "TinyTiM_Lib:RGB_WS2811" H 2575 1975 60  0001 C CNN
 F 3 "" H 2675 1575 60  0001 C CNN
 	1    2675 1575
@@
 F 0 "U203" V 3600 1575 60  0000 C CNN
 F 1 "RGB_WS2811" V 4225 1550 60  0000 C CNN
-F 2 "RGB_WS2811" H 3725 1975 60  0001 C CNN
+F 2 "TinyTiM_Lib:RGB_WS2811" H 3725 1975 60  0001 C CNN
 F 3 "" H 3825 1575 60  0001 C CNN
 	1    3825 1575
@@
 F 0 "U204" V 4750 1550 60  0000 C CNN
 F 1 "RGB_WS2811" V 5375 1550 60  0000 C CNN
-F 2 "RGB_WS2811" H 4875 1975 60  0001 C CNN
+F 2 "TinyTiM_Lib:RGB_WS2811" H 4875 1975 60  0001 C CNN
 F 3 "" H 4975 1575 60  0001 C CNN
 	1    4975 1575
@@
 F 0 "U205" V 5900 1550 60  0000 C CNN
 F 1 "RGB_WS2811" V 6525 1525 60  0000 C CNN
-F 2 "RGB_WS2811" H 6025 1975 60  0001 C CNN
+F 2 "TinyTiM_Lib:RGB_WS2811" H 6025 1975 60  0001 C CNN
 F 3 "" H 6125 1575 60  0001 C CNN
 	1    6125 1575
@@
 F 0 "U206" V 7050 1550 60  0000 C CNN
 F 1 "RGB_WS2811" V 7675 1550 60  0000 C CNN
-F 2 "RGB_WS2811" H 7175 1975 60  0001 C CNN
+F 2 "TinyTiM_Lib:RGB_WS2811" H 7175 1975 60  0001 C CNN
 F 3 "" H 7275 1575 60  0001 C CNN
 	1    7275 1575
@@
 F 0 "U207" V 8200 1550 60  0000 C CNN
 F 1 "RGB_WS2811" V 8825 1550 60  0000 C CNN
-F 2 "RGB_WS2811" H 8325 1975 60  0001 C CNN
+F 2 "TinyTiM_Lib:RGB_WS2811" H 8325 1975 60  0001 C CNN
 F 3 "" H 8425 1575 60  0001 C CNN
 	1    8425 1575
@@
 F 0 "U208" V 9350 1550 60  0000 C CNN
 F 1 "RGB_WS2811" V 9975 1550 60  0000 C CNN
-F 2 "RGB_WS2811" H 9475 1975 60  0001 C CNN
+F 2 "TinyTiM_Lib:RGB_WS2811" H 9475 1975 60  0001 C CNN
 F 3 "" H 9575 1575 60  0001 C CNN
 	1    9575 1575
@@
 F 0 "C217" H 1375 6725 50  0000 L CNN
 F 1 "47u,8V" H 1375 6625 50  0000 L CNN
-F 2 "c_2917" H 1250 6700 50  0001 C CNN
+F 2 "TinyTiM_Lib:c_2917" H 1250 6700 50  0001 C CNN
 F 3 "" H 1250 6750 60  0001 C CNN
 F 4 "CAP ALUM 47UF 8V 20% SMD" H 1250 6950 60  0001 L CNN "Field4"
