File: KiCad/Row_D.sch (KiCad schematic (older format))
At the start: 14 parts, among them U401 RGB_WS2811, U402 RGB_WS2811, U403 RGB_WS2811, U404 RGB_WS2811, U405 RGB_WS2811, U406 RGB_WS2811, U407 RGB_WS2811, U408 RGB_WS2811

Commit message: TinyTiM KiCad work in progress
Parts:
- C401: footprint c_0805 -> TinyTiM_Lib:c_0805
- C417: footprint c_2917 -> TinyTiM_Lib:c_2917
- S401, S402, S403, S404: footprint Screw -> TinyTiM_Lib:Screw
- U401, U402, U403, U404, U405, U406, U407, U408: footprint RGB_WS2811 -> TinyTiM_Lib:RGB_WS2811
Changed lines of the file:
@@
 F 0 "U401" V 1300 1575 60  0000 C CNN
 F 1 "RGB_WS2811" V 1925 1550 60  0000 C CNN
-F 2 "RGB_WS2811" H 1425 1975 60  0001 C CNN
+F 2 "TinyTiM_Lib:RGB_WS2811" H 1425 1975 60  0001 C CNN
 F 3 "" H 1525 1575 60  0001 C CNN
 	1    1525 1575
@@
 F 0 "C401" H 1825 2700 50  0000 L CNN
 F 1 "100n" H 1825 2500 50  0000 L CNN
-F 2 "c_0805" H 1800 2600 50  0001 C CNN
+F 2 "TinyTiM_Lib:c_0805" H 1800 2600 50  0001 C CNN
 F 3 "" H 1800 2600 60  0001 C CNN
 F 4 "CAP CER 0.1UF 25V 10% X7R 0805" H 1800 2800 60  0001 L CNN "Field4"
@@
 F 0 "U402" V 2450 1575 60  0000 C CNN
 F 1 "RGB_WS2811" V 3075 1550 60  0000 C CNN
-F 2 "RGB_WS2811" H 2575 1975 60  0001 C CNN
+F 2 "TinyTiM_Lib:RGB_WS2811" H 2575 1975 60  0001 C CNN
 F 3 "" H 2675 1575 60  0001 C CNN
 	1    2675 1575
@@
 F 0 "U403" V 3600 1575 60  0000 C CNN
 F 1 "RGB_WS2811" V 4225 1550 60  0000 C CNN
-F 2 "RGB_WS2811" H 3725 1975 60  0001 C CNN
+F 2 "TinyTiM_Lib:RGB_WS2811" H 3725 1975 60  0001 C CNN
 F 3 "" H 3825 1575 60  0001 C CNN
 	1    3825 1575
@@
 F 0 "U404" V 4750 1550 60  0000 C CNN
 F 1 "RGB_WS2811" V 5375 1550 60  0000 C CNN
-F 2 "RGB_WS2811" H 4875 1975 60  0001 C CNN
+F 2 "TinyTiM_Lib:RGB_WS2811" H 4875 1975 60  0001 C CNN
 F 3 "" H 4975 1575 60  0001 C CNN
 	1    4975 1575
@@
 F 0 "U405" V 5900 1550 60  0000 C CNN
 F 1 "RGB_WS2811" V 6525 1525 60  0000 C CNN
-F 2 "RGB_WS2811" H 6025 1975 60  0001 C CNN
+F 2 "TinyTiM_Lib:RGB_WS2811" H 6025 1975 60  0001 C CNN
 F 3 "" H 6125 1575 60  0001 C CNN
 	1    6125 1575
@@
 F 0 "U406" V 7050 1550 60  0000 C CNN
 F 1 "RGB_WS2811" V 7675 1550 60  0000 C CNN
-F 2 "RGB_WS2811" H 7175 1975 60  0001 C CNN
+F 2 "TinyTiM_Lib:RGB_WS2811" H 7175 1975 60  0001 C CNN
 F 3 "" H 7275 1575 60  0001 C CNN
 	1    7275 1575
@@
 F 0 "U407" V 8200 1550 60  0000 C CNN
 F 1 "RGB_WS2811" V 8825 1550 60  0000 C CNN
-F 2 "RGB_WS2811" H 8325 1975 60  0001 C CNN
+F 2 "TinyTiM_Lib:RGB_WS2811" H 8325 1975 60  0001 C CNN
 F 3 "" H 8425 1575 60  0001 C CNN
 	1    8425 1575
@@
 F 0 "U408" V 9350 1550 60  0000 C CNN
 F 1 "RGB_WS2811" V 9975 1550 60  0000 C CNN
-F 2 "RGB_WS2811" H 9475 1975 60  0001 C CNN
+F 2 "TinyTiM_Lib:RGB_WS2811" H 9475 1975 60  0001 C CNN
 F 3 "" H 9575 1575 60  0001 C CNN
 	1    9575 1575
@@
 F 0 "S401" V 5380 6650 40  0000 L CNN
 F 1 "CONN_1" H 5300 6705 30  0001 C CNN
-F 2 "Screw" H 5300 6805 30  0001 C CNN
+F 2 "TinyTiM_Lib:Screw" H 5300 6805 30  0001 C CNN
 F 3 "" H 5300 6650 60  0001 C CNN
 	1    5300 6650
@@
 F 0 "S402" V 5580 6650 40  0000 L CNN
 F 1 "CONN_1" H 5500 6705 30  0001 C CNN
-F 2 "Screw" H 5500 6805 30  0001 C CNN
+F 2 "TinyTiM_Lib:Screw" H 5500 6805 30  0001 C CNN
 F 3 "" H 5500 6650 60  0001 C CNN
 	1    5500 6650
@@
 F 0 "S403" V 5780 6650 40  0000 L CNN
 F 1 "CONN_1" H 5700 6705 30  0001 C CNN
-F 2 "Screw" H 5700 6805 30  0001 C CNN
+F 2 "TinyTiM_Lib:Screw" H 5700 6805 30  0001 C CNN
 F 3 "" H 5700 6650 60  0001 C CNN
 	1    5700 6650
@@
 F 0 "S404" V 5980 6650 40  0000 L CNN
 F 1 "CONN_1" H 5900 6705 30  0001 C CNN
-F 2 "Screw" H 5900 6805 30  0001 C CNN
+F 2 "TinyTiM_Lib:Screw" H 5900 6805 30  0001 C CNN
 F 3 "" H 5900 6650 60  0001 C CNN
 	1    5900 6650
@@
 F 0 "C417" H 1375 6725 50  0000 L CNN
 F 1 "47u,8V" H 1375 6625 50  0000 L CNN
-F 2 "c_2917" H 1250 6700 50  0001 C CNN
+F 2 "TinyTiM_Lib:c_2917" H 1250 6700 50  0001 C CNN
 F 3 "" H 1250 6750 60  0001 C CNN
 F 4 "CAP ALUM 47UF 8V 20% SMD" H 1250 6950 60  0001 L CNN "Field4"

Commit message: TinyTiM KiCad work in progress
Parts:
- removed S403, S404: CONN_1, TinyTiM_Lib:Screw, symbol CONN_1
Connections:
- no-connect marks 12 -> 10
Changed lines of the file:
@@
-	0    -1   -1   0
-$EndComp
-$Comp
-L CONN_1 S403
-U 1 1 5118AB6F
-P 5700 6650
-F 0 "S403" V 5780 6650 40  0000 L CNN
-F 1 "CONN_1" H 5700 6705 30  0001 C CNN
-F 2 "TinyTiM_Lib:Screw" H 5700 6805 30  0001 C CNN
-F 3 "" H 5700 6650 60  0001 C CNN
-	1    5700 6650
-	0    -1   -1   0
-$EndComp
-$Comp
-L CONN_1 S404
-U 1 1 5118AB65
-P 5900 6650
-F 0 "S404" V 5980 6650 40  0000 L CNN
-F 1 "CONN_1" H 5900 6705 30  0001 C CNN
-F 2 "TinyTiM_Lib:Screw" H 5900 6805 30  0001 C CNN
-F 3 "" H 5900 6650 60  0001 C CNN
-	1    5900 6650
 	0    -1   -1   0
 $EndComp
 NoConn ~ 5300 6800
 NoConn ~ 5500 6800
-NoConn ~ 5700 6800
-NoConn ~ 5900 6800
 Text Notes 5200 7000 0    60   ~ 0
 Mounting Screws
