File: KiCad/Row_G.sch (KiCad schematic (older format))
At the start: 10 parts, among them U701 RGB_WS2811, U702 RGB_WS2811, U703 RGB_WS2811, U704 RGB_WS2811, U705 RGB_WS2811, U706 RGB_WS2811, U707 RGB_WS2811, U708 RGB_WS2811

Commit message: TinyTiM KiCad work in progress
Parts:
- C701: footprint c_0805 -> TinyTiM_Lib:c_0805
- C717: footprint c_2917 -> TinyTiM_Lib:c_2917
- U701, U702, U703, U704, U705, U706, U707, U708: footprint RGB_WS2811 -> TinyTiM_Lib:RGB_WS2811
Changed lines of the file:
@@
 F 0 "U701" V 1300 1575 60  0000 C CNN
 F 1 "RGB_WS2811" V 1925 1550 60  0000 C CNN
-F 2 "RGB_WS2811" H 1425 1975 60  0001 C CNN
+F 2 "TinyTiM_Lib:RGB_WS2811" H 1425 1975 60  0001 C CNN
 F 3 "" H 1525 1575 60  0001 C CNN
 	1    1525 1575
@@
 F 0 "C701" H 1825 2700 50  0000 L CNN
 F 1 "100n" H 1825 2500 50  0000 L CNN
-F 2 "c_0805" H 1800 2600 50  0001 C CNN
+F 2 "TinyTiM_Lib:c_0805" H 1800 2600 50  0001 C CNN
 F 3 "" H 1800 2600 60  0001 C CNN
 F 4 "CAP CER 0.1UF 25V 10% X7R 0805" H 1800 2800 60  0001 L CNN "Field4"
@@
 F 0 "U702" V 2450 1575 60  0000 C CNN
 F 1 "RGB_WS2811" V 3075 1550 60  0000 C CNN
-F 2 "RGB_WS2811" H 2575 1975 60  0001 C CNN
+F 2 "TinyTiM_Lib:RGB_WS2811" H 2575 1975 60  0001 C CNN
 F 3 "" H 2675 1575 60  0001 C CNN
 	1    2675 1575
@@
 F 0 "U703" V 3600 1575 60  0000 C CNN
 F 1 "RGB_WS2811" V 4225 1550 60  0000 C CNN
-F 2 "RGB_WS2811" H 3725 1975 60  0001 C CNN
+F 2 "TinyTiM_Lib:RGB_WS2811" H 3725 1975 60  0001 C CNN
 F 3 "" H 3825 1575 60  0001 C CNN
 	1    3825 1575
@@
 F 0 "U704" V 4750 1550 60  0000 C CNN
 F 1 "RGB_WS2811" V 5375 1550 60  0000 C CNN
-F 2 "RGB_WS2811" H 4875 1975 60  0001 C CNN
+F 2 "TinyTiM_Lib:RGB_WS2811" H 4875 1975 60  0001 C CNN
 F 3 "" H 4975 1575 60  0001 C CNN
 	1    4975 1575
@@
 F 0 "U705" V 5900 1550 60  0000 C CNN
 F 1 "RGB_WS2811" V 6525 1525 60  0000 C CNN
-F 2 "RGB_WS2811" H 6025 1975 60  0001 C CNN
+F 2 "TinyTiM_Lib:RGB_WS2811" H 6025 1975 60  0001 C CNN
 F 3 "" H 6125 1575 60  0001 C CNN
 	1    6125 1575
@@
 F 0 "U706" V 7050 1550 60  0000 C CNN
 F 1 "RGB_WS2811" V 7675 1550 60  0000 C CNN
-F 2 "RGB_WS2811" H 7175 1975 60  0001 C CNN
+F 2 "TinyTiM_Lib:RGB_WS2811" H 7175 1975 60  0001 C CNN
 F 3 "" H 7275 1575 60  0001 C CNN
 	1    7275 1575
@@
 F 0 "U707" V 8200 1550 60  0000 C CNN
 F 1 "RGB_WS2811" V 8825 1550 60  0000 C CNN
-F 2 "RGB_WS2811" H 8325 1975 60  0001 C CNN
+F 2 "TinyTiM_Lib:RGB_WS2811" H 8325 1975 60  0001 C CNN
 F 3 "" H 8425 1575 60  0001 C CNN
 	1    8425 1575
@@
 F 0 "U708" V 9350 1550 60  0000 C CNN
 F 1 "RGB_WS2811" V 9975 1550 60  0000 C CNN
-F 2 "RGB_WS2811" H 9475 1975 60  0001 C CNN
+F 2 "TinyTiM_Lib:RGB_WS2811" H 9475 1975 60  0001 C CNN
 F 3 "" H 9575 1575 60  0001 C CNN
 	1    9575 1575
@@
 F 0 "C717" H 1375 6725 50  0000 L CNN
 F 1 "47u,8V" H 1375 6625 50  0000 L CNN
-F 2 "c_2917" H 1250 6700 50  0001 C CNN
+F 2 "TinyTiM_Lib:c_2917" H 1250 6700 50  0001 C CNN
 F 3 "" H 1250 6750 60  0001 C CNN
 F 4 "CAP ALUM 47UF 8V 20% SMD" H 1250 6950 60  0001 L CNN "Field4"
