File: KiCad/Row_H.sch (KiCad schematic (older format))
At the start: 14 parts, among them U801 RGB_WS2811, U802 RGB_WS2811, U803 RGB_WS2811, U804 RGB_WS2811, U805 RGB_WS2811, U806 RGB_WS2811, U807 RGB_WS2811, U808 RGB_WS2811

Commit message: TinyTiM KiCad work in progress
Parts:
- C801: footprint c_0805 -> TinyTiM_Lib:c_0805
- C817: footprint c_2917 -> TinyTiM_Lib:c_2917
- S801, S802, S803, S804: footprint Screw -> TinyTiM_Lib:Screw
- U801, U802, U803, U804, U805, U806, U807, U808: footprint RGB_WS2811 -> TinyTiM_Lib:RGB_WS2811
Changed lines of the file:
@@
 F 0 "U801" V 1300 1575 60  0000 C CNN
 F 1 "RGB_WS2811" V 1925 1550 60  0000 C CNN
-F 2 "RGB_WS2811" H 1425 1975 60  0001 C CNN
+F 2 "TinyTiM_Lib:RGB_WS2811" H 1425 1975 60  0001 C CNN
 F 3 "" H 1525 1575 60  0001 C CNN
 	1    1525 1575
@@
 F 0 "C801" H 1825 2700 50  0000 L CNN
 F 1 "100n" H 1825 2500 50  0000 L CNN
-F 2 "c_0805" H 1800 2600 50  0001 C CNN
+F 2 "TinyTiM_Lib:c_0805" H 1800 2600 50  0001 C CNN
 F 3 "" H 1800 2600 60  0001 C CNN
 F 4 "CAP CER 0.1UF 25V 10% X7R 0805" H 1800 2800 60  0001 L CNN "Field4"
@@
 F 0 "U802" V 2450 1575 60  0000 C CNN
 F 1 "RGB_WS2811" V 3075 1550 60  0000 C CNN
-F 2 "RGB_WS2811" H 2575 1975 60  0001 C CNN
+F 2 "TinyTiM_Lib:RGB_WS2811" H 2575 1975 60  0001 C CNN
 F 3 "" H 2675 1575 60  0001 C CNN
 	1    2675 1575
@@
 F 0 "U803" V 3600 1575 60  0000 C CNN
 F 1 "RGB_WS2811" V 4225 1550 60  0000 C CNN
-F 2 "RGB_WS2811" H 3725 1975 60  0001 C CNN
+F 2 "TinyTiM_Lib:RGB_WS2811" H 3725 1975 60  0001 C CNN
 F 3 "" H 3825 1575 60  0001 C CNN
 	1    3825 1575
@@
 F 0 "U804" V 4750 1550 60  0000 C CNN
 F 1 "RGB_WS2811" V 5375 1550 60  0000 C CNN
-F 2 "RGB_WS2811" H 4875 1975 60  0001 C CNN
+F 2 "TinyTiM_Lib:RGB_WS2811" H 4875 1975 60  0001 C CNN
 F 3 "" H 4975 1575 60  0001 C CNN
 	1    4975 1575
@@
 F 0 "U805" V 5900 1550 60  0000 C CNN
 F 1 "RGB_WS2811" V 6525 1525 60  0000 C CNN
-F 2 "RGB_WS2811" H 6025 1975 60  0001 C CNN
+F 2 "TinyTiM_Lib:RGB_WS2811" H 6025 1975 60  0001 C CNN
 F 3 "" H 6125 1575 60  0001 C CNN
 	1    6125 1575
@@
 F 0 "U806" V 7050 1550 60  0000 C CNN
 F 1 "RGB_WS2811" V 7675 1550 60  0000 C CNN
-F 2 "RGB_WS2811" H 7175 1975 60  0001 C CNN
+F 2 "TinyTiM_Lib:RGB_WS2811" H 7175 1975 60  0001 C CNN
 F 3 "" H 7275 1575 60  0001 C CNN
 	1    7275 1575
@@
 F 0 "U807" V 8200 1550 60  0000 C CNN
 F 1 "RGB_WS2811" V 8825 1550 60  0000 C CNN
-F 2 "RGB_WS2811" H 8325 1975 60  0001 C CNN
+F 2 "TinyTiM_Lib:RGB_WS2811" H 8325 1975 60  0001 C CNN
 F 3 "" H 8425 1575 60  0001 C CNN
 	1    8425 1575
@@
 F 0 "U808" V 9350 1550 60  0000 C CNN
 F 1 "RGB_WS2811" V 9975 1550 60  0000 C CNN
-F 2 "RGB_WS2811" H 9475 1975 60  0001 C CNN
+F 2 "TinyTiM_Lib:RGB_WS2811" H 9475 1975 60  0001 C CNN
 F 3 "" H 9575 1575 60  0001 C CNN
 	1    9575 1575
@@
 F 0 "S801" V 5380 6650 40  0000 L CNN
 F 1 "CONN_1" H 5300 6705 30  0001 C CNN
-F 2 "Screw" H 5300 6805 30  0001 C CNN
+F 2 "TinyTiM_Lib:Screw" H 5300 6805 30  0001 C CNN
 F 3 "" H 5300 6650 60  0001 C CNN
 	1    5300 6650
@@
 F 0 "S802" V 5580 6650 40  0000 L CNN
 F 1 "CONN_1" H 5500 6705 30  0001 C CNN
-F 2 "Screw" H 5500 6805 30  0001 C CNN
+F 2 "TinyTiM_Lib:Screw" H 5500 6805 30  0001 C CNN
 F 3 "" H 5500 6650 60  0001 C CNN
 	1    5500 6650
@@
 F 0 "S803" V 5780 6650 40  0000 L CNN
 F 1 "CONN_1" H 5700 6705 30  0001 C CNN
-F 2 "Screw" H 5700 6805 30  0001 C CNN
+F 2 "TinyTiM_Lib:Screw" H 5700 6805 30  0001 C CNN
 F 3 "" H 5700 6650 60  0001 C CNN
 	1    5700 6650
@@
 F 0 "S804" V 5980 6650 40  0000 L CNN
 F 1 "CONN_1" H 5900 6705 30  0001 C CNN
-F 2 "Screw" H 5900 6805 30  0001 C CNN
+F 2 "TinyTiM_Lib:Screw" H 5900 6805 30  0001 C CNN
 F 3 "" H 5900 6650 60  0001 C CNN
 	1    5900 6650
@@
 F 0 "C817" H 1375 6725 50  0000 L CNN
 F 1 "47u,8V" H 1375 6625 50  0000 L CNN
-F 2 "c_2917" H 1250 6700 50  0001 C CNN
+F 2 "TinyTiM_Lib:c_2917" H 1250 6700 50  0001 C CNN
 F 3 "" H 1250 6750 60  0001 C CNN
 F 4 "CAP ALUM 47UF 8V 20% SMD" H 1250 6950 60  0001 L CNN "Field4"
