File: KiCad/TinyTiM.sch (KiCad schematic (older format))
At the start: 16 parts, among them P1 PWR_W, P125 G>H, P126 F>G, P127 E>F, P128 D>E, P129 C>D, P130 B>C, P131 A>B, P2 PWR_E, P3 Data_In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

Commit message: minor mods to silk legend. Final, ready for prototyping
Parts:
- removed PCB101: CONN_1, TinyTiM_Lib:PCB, symbol CONN_1
Connections:
- no-connect marks 3 -> 2
Changed lines of the file:
@@
 01 31 04 0B 88 21 58 40 0C C1 02 62 08 16 10 43 B0 80 18 82 05 C4 10 2C 20 86 60 01 31 04 0B 88
 21 58 40 0C C1 02 62 08 16 10 43 B0 80 18 82 05 C4 10 2C 20 86 60 01 31 04 0B 88 21 58 40 0C C1
-02 62 7C 03 3D 79 5E 0E 30 13 47 E7 00 00 00 00 49 45 4E 44 AE 42 60 82 F8
+02 62 7C 03 3D 79 5E 0E 30 13 47 E7 00 00 00 00 49 45 4E 44 AE 42 60 82 91
 EndData
 $EndBitmap
@@
 C1 ED 35 72 E0 F7 FB FF F1 1F FF F1 9F FF F9 9F C7 C7 C7 73 1A 9F 2B 70 38 1C FB F6 ED 3B 79 F2
 E4 23 8F 3C 52 B0 F1 D9 2E 76 F1 FF 03 17 ED 19 47 28 92 59 FB 00 00 00 00 49 45 4E 44 AE 42 60
-82 CF
+82 3D
 EndData
 $EndBitmap
@@
 	0    -1   -1   0
 $EndComp
-NoConn ~ 1300 7500
-$Comp
-L CONN_1 PCB101
-U 1 1 5118E269
-P 1300 7350
-F 0 "PCB101" H 1380 7350 40  0000 L CNN
-F 1 "CONN_1" H 1300 7405 30  0001 C CNN
-F 2 "TinyTiM_Lib:PCB" H 1175 7400 30  0001 C CNN
-F 3 "" H 1300 7350 60  0001 C CNN
-	1    1300 7350
-	0    -1   -1   0
-$EndComp
