File: KiCad/rev2/Row_A.sch (KiCad schematic (older format))
At the start: 14 parts, among them U101 RGB_WS2811, U102 RGB_WS2811, U103 RGB_WS2811, U104 RGB_WS2811, U105 RGB_WS2811, U106 RGB_WS2811, U107 RGB_WS2811, U108 RGB_WS2811

Commit message: TinyTiM rev2 work in progress, schematic complete
Parts:
- U101, U102, U103, U104, U105, U106, U107, U108: value RGB_WS2811 -> RGB_WS2811B; footprint TinyTiM_Lib:RGB_WS2811 -> TinyTiM_Lib:RGB_WS2811B; symbol RGB_WS2811 -> RGB_WS2811B
Connections:
- net 5V: now also U101.1 (VDD), U102.1 (VDD), U103.1 (VDD), U104.1 (VDD), U105.1 (VDD), U106.1 (VDD), U107.1 (VDD), U108.1 (VDD); no longer U101.3 (VCC), U101.5 (VDD), U102.3 (VCC), U102.5 (VDD), U103.3 (VCC), U103.5 (VDD), U104.3 (VCC), U104.5 (VDD), U105.3 (VCC), U105.5 (VDD), U106.3 (VCC), U106.5 (VDD), U107.3 (VCC), U107.5 (VDD), U108.3 (VCC), U108.5 (VDD)
- net A_02: now also U101.2 (DO), U102.4 (DI); no longer U101.1 (DO), U102.2 (DI)
- net A_03: now also U102.2 (DO), U103.4 (DI); no longer U102.1 (DO), U103.2 (DI)
- net A_04: now also U103.2 (DO), U104.4 (DI); no longer U103.1 (DO), U104.2 (DI)
- net A_05: now also U104.2 (DO), U105.4 (DI); no longer U104.1 (DO), U105.2 (DI)
- net A_06: now also U105.2 (DO), U106.4 (DI); no longer U105.1 (DO), U106.2 (DI)
- net A_07: now also U106.2 (DO), U107.4 (DI); no longer U106.1 (DO), U107.2 (DI)
- net A_08: now also U107.2 (DO), U108.4 (DI); no longer U107.1 (DO), U108.2 (DI)
- net DI_A: now also U101.4 (DI); no longer U101.2 (DI)
- net DO_A: now also U108.2 (DO); no longer U108.1 (DO)
- net GND: now also U101.3 (VSS), U102.3 (VSS), U103.3 (VSS), U104.3 (VSS), U105.3 (VSS), U106.3 (VSS), U107.3 (VSS), U108.3 (VSS); no longer U101.6 (VSS), U102.6 (VSS), U103.6 (VSS), U104.6 (VSS), U105.6 (VSS), U106.6 (VSS), U107.6 (VSS), U108.6 (VSS)
- no-connect marks 12 -> 4
Changed lines of the file:
@@
 Text HLabel 950  900  0    60   Input ~ 0
 DI_A
-Text HLabel 950  750  0    60   Input ~ 0
+Text HLabel 950  2850 0    60   Input ~ 0
 5V
 $Comp
-L RGB_WS2811 U101
+L RGB_WS2811B U101
 U 1 1 51189846
 P 1525 1575
 F 0 "U101" V 1300 1575 60  0000 C CNN
-F 1 "RGB_WS2811" V 1925 1550 60  0000 C CNN
-F 2 "TinyTiM_Lib:RGB_WS2811" H 1425 1975 60  0001 C CNN
+F 1 "RGB_WS2811B" V 1925 1550 60  0000 C CNN
+F 2 "TinyTiM_Lib:RGB_WS2811B" H 1425 1975 60  0001 C CNN
 F 3 "" H 1525 1575 60  0001 C CNN
 	1    1525 1575
 	1    0    0    -1
 $EndComp
-NoConn ~ 1400 2200
-NoConn ~ 2550 2200
-NoConn ~ 3700 2200
-NoConn ~ 4850 2200
-NoConn ~ 6000 2200
-NoConn ~ 7150 2200
-NoConn ~ 8300 2200
-NoConn ~ 9450 2200
-Text Label 950  750  0    60   ~ 0
-5V
 Text Label 950  2350 0    60   ~ 0
 GND
@@
 $EndComp
 $Comp
-L RGB_WS2811 U102
+L RGB_WS2811B U102
 U 1 1 5118AB0C
 P 2675 1575
 F 0 "U102" V 2450 1575 60  0000 C CNN
-F 1 "RGB_WS2811" V 3075 1550 60  0000 C CNN
-F 2 "TinyTiM_Lib:RGB_WS2811" H 2575 1975 60  0001 C CNN
+F 1 "RGB_WS2811B" V 3075 1550 60  0000 C CNN
+F 2 "TinyTiM_Lib:RGB_WS2811B" H 2575 1975 60  0001 C CNN
 F 3 "" H 2675 1575 60  0001 C CNN
 	1    2675 1575
@@
 $EndComp
 $Comp
-L RGB_WS2811 U103
+L RGB_WS2811B U103
 U 1 1 5118AB00
 P 3825 1575
 F 0 "U103" V 3600 1575 60  0000 C CNN
-F 1 "RGB_WS2811" V 4225 1550 60  0000 C CNN
-F 2 "TinyTiM_Lib:RGB_WS2811" H 3725 1975 60  0001 C CNN
+F 1 "RGB_WS2811B" V 4225 1550 60  0000 C CNN
+F 2 "TinyTiM_Lib:RGB_WS2811B" H 3725 1975 60  0001 C CNN
 F 3 "" H 3825 1575 60  0001 C CNN
 	1    3825 1575
@@
 $EndComp
 $Comp
-L RGB_WS2811 U104
+L RGB_WS2811B U104
 U 1 1 5118AB8D
 P 4975 1575
 F 0 "U104" V 4750 1550 60  0000 C CNN
-F 1 "RGB_WS2811" V 5375 1550 60  0000 C CNN
-F 2 "TinyTiM_Lib:RGB_WS2811" H 4875 1975 60  0001 C CNN
+F 1 "RGB_WS2811B" V 5375 1550 60  0000 C CNN
+F 2 "TinyTiM_Lib:RGB_WS2811B" H 4875 1975 60  0001 C CNN
 F 3 "" H 4975 1575 60  0001 C CNN
 	1    4975 1575
@@
 $EndComp
 $Comp
-L RGB_WS2811 U105
+L RGB_WS2811B U105
 U 1 1 5118AAFC
 P 6125 1575
 F 0 "U105" V 5900 1550 60  0000 C CNN
-F 1 "RGB_WS2811" V 6525 1525 60  0000 C CNN
-F 2 "TinyTiM_Lib:RGB_WS2811" H 6025 1975 60  0001 C CNN
+F 1 "RGB_WS2811B" V 6525 1525 60  0000 C CNN
+F 2 "TinyTiM_Lib:RGB_WS2811B" H 6025 1975 60  0001 C CNN
 F 3 "" H 6125 1575 60  0001 C CNN
 	1    6125 1575
@@
 $EndComp
 $Comp
-L RGB_WS2811 U106
+L RGB_WS2811B U106
 U 1 1 5118AAF2
 P 7275 1575
 F 0 "U106" V 7050 1550 60  0000 C CNN
-F 1 "RGB_WS2811" V 7675 1550 60  0000 C CNN
-F 2 "TinyTiM_Lib:RGB_WS2811" H 7175 1975 60  0001 C CNN
+F 1 "RGB_WS2811B" V 7675 1550 60  0000 C CNN
+F 2 "TinyTiM_Lib:RGB_WS2811B" H 7175 1975 60  0001 C CNN
 F 3 "" H 7275 1575 60  0001 C CNN
 	1    7275 1575
@@
 $EndComp
 $Comp
-L RGB_WS2811 U107
+L RGB_WS2811B U107
 U 1 1 5118AAF0
 P 8425 1575
 F 0 "U107" V 8200 1550 60  0000 C CNN
-F 1 "RGB_WS2811" V 8825 1550 60  0000 C CNN
-F 2 "TinyTiM_Lib:RGB_WS2811" H 8325 1975 60  0001 C CNN
+F 1 "RGB_WS2811B" V 8825 1550 60  0000 C CNN
+F 2 "TinyTiM_Lib:RGB_WS2811B" H 8325 1975 60  0001 C CNN
 F 3 "" H 8425 1575 60  0001 C CNN
 	1    8425 1575
@@
 $EndComp
 $Comp
-L RGB_WS2811 U108
+L RGB_WS2811B U108
 U 1 1 5118AAE5
 P 9575 1575
 F 0 "U108" V 9350 1550 60  0000 C CNN
-F 1 "RGB_WS2811" V 9975 1550 60  0000 C CNN
-F 2 "TinyTiM_Lib:RGB_WS2811" H 9475 1975 60  0001 C CNN
+F 1 "RGB_WS2811B" V 9975 1550 60  0000 C CNN
+F 2 "TinyTiM_Lib:RGB_WS2811B" H 9475 1975 60  0001 C CNN
 F 3 "" H 9575 1575 60  0001 C CNN
 	1    9575 1575
@@
 	1150 2400 1150 2350
 Wire Wire Line
-	1400 1000 1400 750
-Wire Wire Line
 	9850 2350 9850 2200
 Wire Wire Line
@@
 Wire Wire Line
 	950  2350 9850 2350
-Connection ~ 1400 750
-Wire Wire Line
-	950  750  9450 750
 Connection ~ 4100 2350
 Connection ~ 6400 2350
@@
 Wire Wire Line
 	1600 2850 1600 2200
-Connection ~ 2550 750
-Wire Wire Line
-	2550 750  2550 1000
-Connection ~ 4850 750
-Wire Wire Line
-	4850 750  4850 1000
-Connection ~ 7150 750
-Wire Wire Line
-	7150 750  7150 1000
-Wire Wire Line
-	9450 750  9450 1000
-Wire Wire Line
-	8300 1000 8300 750
-Connection ~ 8300 750
-Wire Wire Line
-	6000 750  6000 1000
-Connection ~ 6000 750
-Wire Wire Line
-	3700 750  3700 1000
-Connection ~ 3700 750
 Wire Wire Line
 	8500 2850 8500 2200
