File: KiCad/rev2/Row_B.sch (KiCad schematic (older format))
At the start: 10 parts, among them U201 RGB_WS2811, U202 RGB_WS2811, U203 RGB_WS2811, U204 RGB_WS2811, U205 RGB_WS2811, U206 RGB_WS2811, U207 RGB_WS2811, U208 RGB_WS2811

Commit message: TinyTiM rev2 work in progress, schematic complete
Parts:
- U201, U202, U203, U204, U205, U206, U207, U208: value RGB_WS2811 -> RGB_WS2811B; footprint TinyTiM_Lib:RGB_WS2811 -> TinyTiM_Lib:RGB_WS2811B; symbol RGB_WS2811 -> RGB_WS2811B
Connections:
- net 5V: now also U201.1 (VDD), U202.1 (VDD), U203.1 (VDD), U204.1 (VDD), U205.1 (VDD), U206.1 (VDD), U207.1 (VDD), U208.1 (VDD); no longer U201.3 (VCC), U201.5 (VDD), U202.3 (VCC), U202.5 (VDD), U203.3 (VCC), U203.5 (VDD), U204.3 (VCC), U204.5 (VDD), U205.3 (VCC), U205.5 (VDD), U206.3 (VCC), U206.5 (VDD), U207.3 (VCC), U207.5 (VDD), U208.3 (VCC), U208.5 (VDD)
- net B_02: now also U201.2 (DO), U202.4 (DI); no longer U201.1 (DO), U202.2 (DI)
- net B_03: now also U202.2 (DO), U203.4 (DI); no longer U202.1 (DO), U203.2 (DI)
- net B_04: now also U203.2 (DO), U204.4 (DI); no longer U203.1 (DO), U204.2 (DI)
- net B_05: now also U204.2 (DO), U205.4 (DI); no longer U204.1 (DO), U205.2 (DI)
- net B_06: now also U205.2 (DO), U206.4 (DI); no longer U205.1 (DO), U206.2 (DI)
- net B_07: now also U206.2 (DO), U207.4 (DI); no longer U206.1 (DO), U207.2 (DI)
- net B_08: now also U207.2 (DO), U208.4 (DI); no longer U207.1 (DO), U208.2 (DI)
- net DI_B: now also U201.4 (DI); no longer U201.2 (DI)
- net DO_B: now also U208.2 (DO); no longer U208.1 (DO)
- net GND: now also U201.3 (VSS), U202.3 (VSS), U203.3 (VSS), U204.3 (VSS), U205.3 (VSS), U206.3 (VSS), U207.3 (VSS), U208.3 (VSS); no longer U201.6 (VSS), U202.6 (VSS), U203.6 (VSS), U204.6 (VSS), U205.6 (VSS), U206.6 (VSS), U207.6 (VSS), U208.6 (VSS)
- no-connect marks 8 -> 0
Changed lines of the file:
@@
 Text HLabel 950  900  0    60   Input ~ 0
 DI_B
-Text HLabel 950  750  0    60   Input ~ 0
+Text HLabel 950  2850 0    60   Input ~ 0
 5V
 $Comp
-L RGB_WS2811 U201
+L RGB_WS2811B U201
 U 1 1 5118ABBA
 P 1525 1575
 F 0 "U201" V 1300 1575 60  0000 C CNN
-F 1 "RGB_WS2811" V 1925 1550 60  0000 C CNN
-F 2 "TinyTiM_Lib:RGB_WS2811" H 1425 1975 60  0001 C CNN
+F 1 "RGB_WS2811B" V 1925 1550 60  0000 C CNN
+F 2 "TinyTiM_Lib:RGB_WS2811B" H 1425 1975 60  0001 C CNN
 F 3 "" H 1525 1575 60  0001 C CNN
 	1    1525 1575
 	1    0    0    -1
 $EndComp
-NoConn ~ 1400 2200
-NoConn ~ 2550 2200
-NoConn ~ 3700 2200
-NoConn ~ 4850 2200
-NoConn ~ 6000 2200
-NoConn ~ 7150 2200
-NoConn ~ 8300 2200
-NoConn ~ 9450 2200
-Text Label 950  750  0    60   ~ 0
-5V
 Text Label 950  2350 0    60   ~ 0
 GND
@@
 $EndComp
 $Comp
-L RGB_WS2811 U202
+L RGB_WS2811B U202
 U 1 1 5116894B
 P 2675 1575
 F 0 "U202" V 2450 1575 60  0000 C CNN
-F 1 "RGB_WS2811" V 3075 1550 60  0000 C CNN
-F 2 "TinyTiM_Lib:RGB_WS2811" H 2575 1975 60  0001 C CNN
+F 1 "RGB_WS2811B" V 3075 1550 60  0000 C CNN
+F 2 "TinyTiM_Lib:RGB_WS2811B" H 2575 1975 60  0001 C CNN
 F 3 "" H 2675 1575 60  0001 C CNN
 	1    2675 1575
@@
 $EndComp
 $Comp
-L RGB_WS2811 U203
+L RGB_WS2811B U203
 U 1 1 5118AB01
 P 3825 1575
 F 0 "U203" V 3600 1575 60  0000 C CNN
-F 1 "RGB_WS2811" V 4225 1550 60  0000 C CNN
-F 2 "TinyTiM_Lib:RGB_WS2811" H 3725 1975 60  0001 C CNN
+F 1 "RGB_WS2811B" V 4225 1550 60  0000 C CNN
+F 2 "TinyTiM_Lib:RGB_WS2811B" H 3725 1975 60  0001 C CNN
 F 3 "" H 3825 1575 60  0001 C CNN
 	1    3825 1575
@@
 $EndComp
 $Comp
-L RGB_WS2811 U204
+L RGB_WS2811B U204
 U 1 1 5118AB90
 P 4975 1575
 F 0 "U204" V 4750 1550 60  0000 C CNN
-F 1 "RGB_WS2811" V 5375 1550 60  0000 C CNN
-F 2 "TinyTiM_Lib:RGB_WS2811" H 4875 1975 60  0001 C CNN
+F 1 "RGB_WS2811B" V 5375 1550 60  0000 C CNN
+F 2 "TinyTiM_Lib:RGB_WS2811B" H 4875 1975 60  0001 C CNN
 F 3 "" H 4975 1575 60  0001 C CNN
 	1    4975 1575
@@
 $EndComp
 $Comp
-L RGB_WS2811 U205
+L RGB_WS2811B U205
 U 1 1 5118AAFB
 P 6125 1575
 F 0 "U205" V 5900 1550 60  0000 C CNN
-F 1 "RGB_WS2811" V 6525 1525 60  0000 C CNN
-F 2 "TinyTiM_Lib:RGB_WS2811" H 6025 1975 60  0001 C CNN
+F 1 "RGB_WS2811B" V 6525 1525 60  0000 C CNN
+F 2 "TinyTiM_Lib:RGB_WS2811B" H 6025 1975 60  0001 C CNN
 F 3 "" H 6125 1575 60  0001 C CNN
 	1    6125 1575
@@
 $EndComp
 $Comp
-L RGB_WS2811 U206
+L RGB_WS2811B U206
 U 1 1 5118AAF5
 P 7275 1575
 F 0 "U206" V 7050 1550 60  0000 C CNN
-F 1 "RGB_WS2811" V 7675 1550 60  0000 C CNN
-F 2 "TinyTiM_Lib:RGB_WS2811" H 7175 1975 60  0001 C CNN
+F 1 "RGB_WS2811B" V 7675 1550 60  0000 C CNN
+F 2 "TinyTiM_Lib:RGB_WS2811B" H 7175 1975 60  0001 C CNN
 F 3 "" H 7275 1575 60  0001 C CNN
 	1    7275 1575
@@
 $EndComp
 $Comp
-L RGB_WS2811 U207
+L RGB_WS2811B U207
 U 1 1 5118AAEE
 P 8425 1575
 F 0 "U207" V 8200 1550 60  0000 C CNN
-F 1 "RGB_WS2811" V 8825 1550 60  0000 C CNN
-F 2 "TinyTiM_Lib:RGB_WS2811" H 8325 1975 60  0001 C CNN
+F 1 "RGB_WS2811B" V 8825 1550 60  0000 C CNN
+F 2 "TinyTiM_Lib:RGB_WS2811B" H 8325 1975 60  0001 C CNN
 F 3 "" H 8425 1575 60  0001 C CNN
 	1    8425 1575
@@
 $EndComp
 $Comp
-L RGB_WS2811 U208
+L RGB_WS2811B U208
 U 1 1 5118AAEA
 P 9575 1575
 F 0 "U208" V 9350 1550 60  0000 C CNN
-F 1 "RGB_WS2811" V 9975 1550 60  0000 C CNN
-F 2 "TinyTiM_Lib:RGB_WS2811" H 9475 1975 60  0001 C CNN
+F 1 "RGB_WS2811B" V 9975 1550 60  0000 C CNN
+F 2 "TinyTiM_Lib:RGB_WS2811B" H 9475 1975 60  0001 C CNN
 F 3 "" H 9575 1575 60  0001 C CNN
 	1    9575 1575
@@
 	1150 2400 1150 2350
 Wire Wire Line
-	1400 1000 1400 750
-Wire Wire Line
 	9850 2350 9850 2200
 Wire Wire Line
@@
 Wire Wire Line
 	950  2350 9850 2350
-Connection ~ 1400 750
-Wire Wire Line
-	950  750  9450 750
 Connection ~ 4100 2350
 Connection ~ 6400 2350
@@
 Wire Wire Line
 	1600 2850 1600 2200
-Connection ~ 2550 750
-Wire Wire Line
-	2550 750  2550 1000
-Connection ~ 4850 750
-Wire Wire Line
-	4850 750  4850 1000
-Connection ~ 7150 750
-Wire Wire Line
-	7150 750  7150 1000
-Wire Wire Line
-	9450 750  9450 1000
-Wire Wire Line
-	8300 1000 8300 750
-Connection ~ 8300 750
-Wire Wire Line
-	6000 750  6000 1000
-Connection ~ 6000 750
-Wire Wire Line
-	3700 750  3700 1000
-Connection ~ 3700 750
 Wire Wire Line
 	8500 2850 8500 2200
