File: KiCad/rev2/Row_C.sch (KiCad schematic (older format))
At the start: 10 parts, among them U301 RGB_WS2811, U302 RGB_WS2811, U303 RGB_WS2811, U304 RGB_WS2811, U305 RGB_WS2811, U306 RGB_WS2811, U307 RGB_WS2811, U308 RGB_WS2811

Commit message: TinyTiM rev2 work in progress, schematic complete
Parts:
- U301, U302, U303, U304, U305, U306, U307, U308: value RGB_WS2811 -> RGB_WS2811B; footprint TinyTiM_Lib:RGB_WS2811 -> TinyTiM_Lib:RGB_WS2811B; symbol RGB_WS2811 -> RGB_WS2811B
Connections:
- net 5V: now also U301.1 (VDD), U302.1 (VDD), U303.1 (VDD), U304.1 (VDD), U305.1 (VDD), U306.1 (VDD), U307.1 (VDD), U308.1 (VDD); no longer U301.3 (VCC), U301.5 (VDD), U302.3 (VCC), U302.5 (VDD), U303.3 (VCC), U303.5 (VDD), U304.3 (VCC), U304.5 (VDD), U305.3 (VCC), U305.5 (VDD), U306.3 (VCC), U306.5 (VDD), U307.3 (VCC), U307.5 (VDD), U308.3 (VCC), U308.5 (VDD)
- net C_02: now also U301.2 (DO), U302.4 (DI); no longer U301.1 (DO), U302.2 (DI)
- net C_03: now also U302.2 (DO), U303.4 (DI); no longer U302.1 (DO), U303.2 (DI)
- net C_04: now also U303.2 (DO), U304.4 (DI); no longer U303.1 (DO), U304.2 (DI)
- net C_05: now also U304.2 (DO), U305.4 (DI); no longer U304.1 (DO), U305.2 (DI)
- net C_06: now also U305.2 (DO), U306.4 (DI); no longer U305.1 (DO), U306.2 (DI)
- net C_07: now also U306.2 (DO), U307.4 (DI); no longer U306.1 (DO), U307.2 (DI)
- net C_08: now also U307.2 (DO), U308.4 (DI); no longer U307.1 (DO), U308.2 (DI)
- net DI_C: now also U301.4 (DI); no longer U301.2 (DI)
- net DO_C: now also U308.2 (DO); no longer U308.1 (DO)
- net GND: now also U301.3 (VSS), U302.3 (VSS), U303.3 (VSS), U304.3 (VSS), U305.3 (VSS), U306.3 (VSS), U307.3 (VSS), U308.3 (VSS); no longer U301.6 (VSS), U302.6 (VSS), U303.6 (VSS), U304.6 (VSS), U305.6 (VSS), U306.6 (VSS), U307.6 (VSS), U308.6 (VSS)
- no-connect marks 8 -> 0
Changed lines of the file:
@@
 Text HLabel 950  900  0    60   Input ~ 0
 DI_C
-Text HLabel 950  750  0    60   Input ~ 0
+Text HLabel 950  2850 0    60   Input ~ 0
 5V
 $Comp
-L RGB_WS2811 U301
+L RGB_WS2811B U301
 U 1 1 5118ABB8
 P 1525 1575
 F 0 "U301" V 1300 1575 60  0000 C CNN
-F 1 "RGB_WS2811" V 1925 1550 60  0000 C CNN
-F 2 "TinyTiM_Lib:RGB_WS2811" H 1425 1975 60  0001 C CNN
+F 1 "RGB_WS2811B" V 1925 1550 60  0000 C CNN
+F 2 "TinyTiM_Lib:RGB_WS2811B" H 1425 1975 60  0001 C CNN
 F 3 "" H 1525 1575 60  0001 C CNN
 	1    1525 1575
 	1    0    0    -1
 $EndComp
-NoConn ~ 1400 2200
-NoConn ~ 2550 2200
-NoConn ~ 3700 2200
-NoConn ~ 4850 2200
-NoConn ~ 6000 2200
-NoConn ~ 7150 2200
-NoConn ~ 8300 2200
-NoConn ~ 9450 2200
-Text Label 950  750  0    60   ~ 0
-5V
 Text Label 950  2350 0    60   ~ 0
 GND
@@
 $EndComp
 $Comp
-L RGB_WS2811 U302
+L RGB_WS2811B U302
 U 1 1 5118AB08
 P 2675 1575
 F 0 "U302" V 2450 1575 60  0000 C CNN
-F 1 "RGB_WS2811" V 3075 1550 60  0000 C CNN
-F 2 "TinyTiM_Lib:RGB_WS2811" H 2575 1975 60  0001 C CNN
+F 1 "RGB_WS2811B" V 3075 1550 60  0000 C CNN
+F 2 "TinyTiM_Lib:RGB_WS2811B" H 2575 1975 60  0001 C CNN
 F 3 "" H 2675 1575 60  0001 C CNN
 	1    2675 1575
@@
 $EndComp
 $Comp
-L RGB_WS2811 U303
+L RGB_WS2811B U303
 U 1 1 5118AB02
 P 3825 1575
 F 0 "U303" V 3600 1575 60  0000 C CNN
-F 1 "RGB_WS2811" V 4225 1550 60  0000 C CNN
-F 2 "TinyTiM_Lib:RGB_WS2811" H 3725 1975 60  0001 C CNN
+F 1 "RGB_WS2811B" V 4225 1550 60  0000 C CNN
+F 2 "TinyTiM_Lib:RGB_WS2811B" H 3725 1975 60  0001 C CNN
 F 3 "" H 3825 1575 60  0001 C CNN
 	1    3825 1575
@@
 $EndComp
 $Comp
-L RGB_WS2811 U304
+L RGB_WS2811B U304
 U 1 1 5118AB91
 P 4975 1575
 F 0 "U304" V 4750 1550 60  0000 C CNN
-F 1 "RGB_WS2811" V 5375 1550 60  0000 C CNN
-F 2 "TinyTiM_Lib:RGB_WS2811" H 4875 1975 60  0001 C CNN
+F 1 "RGB_WS2811B" V 5375 1550 60  0000 C CNN
+F 2 "TinyTiM_Lib:RGB_WS2811B" H 4875 1975 60  0001 C CNN
 F 3 "" H 4975 1575 60  0001 C CNN
 	1    4975 1575
@@
 $EndComp
 $Comp
-L RGB_WS2811 U305
+L RGB_WS2811B U305
 U 1 1 5118AAFA
 P 6125 1575
 F 0 "U305" V 5900 1550 60  0000 C CNN
-F 1 "RGB_WS2811" V 6525 1525 60  0000 C CNN
-F 2 "TinyTiM_Lib:RGB_WS2811" H 6025 1975 60  0001 C CNN
+F 1 "RGB_WS2811B" V 6525 1525 60  0000 C CNN
+F 2 "TinyTiM_Lib:RGB_WS2811B" H 6025 1975 60  0001 C CNN
 F 3 "" H 6125 1575 60  0001 C CNN
 	1    6125 1575
@@
 $EndComp
 $Comp
-L RGB_WS2811 U306
+L RGB_WS2811B U306
 U 1 1 5118AAF3
 P 7275 1575
 F 0 "U306" V 7050 1550 60  0000 C CNN
-F 1 "RGB_WS2811" V 7675 1550 60  0000 C CNN
-F 2 "TinyTiM_Lib:RGB_WS2811" H 7175 1975 60  0001 C CNN
+F 1 "RGB_WS2811B" V 7675 1550 60  0000 C CNN
+F 2 "TinyTiM_Lib:RGB_WS2811B" H 7175 1975 60  0001 C CNN
 F 3 "" H 7275 1575 60  0001 C CNN
 	1    7275 1575
@@
 $EndComp
 $Comp
-L RGB_WS2811 U307
+L RGB_WS2811B U307
 U 1 1 5118AAEB
 P 8425 1575
 F 0 "U307" V 8200 1550 60  0000 C CNN
-F 1 "RGB_WS2811" V 8825 1550 60  0000 C CNN
-F 2 "TinyTiM_Lib:RGB_WS2811" H 8325 1975 60  0001 C CNN
+F 1 "RGB_WS2811B" V 8825 1550 60  0000 C CNN
+F 2 "TinyTiM_Lib:RGB_WS2811B" H 8325 1975 60  0001 C CNN
 F 3 "" H 8425 1575 60  0001 C CNN
 	1    8425 1575
@@
 $EndComp
 $Comp
-L RGB_WS2811 U308
+L RGB_WS2811B U308
 U 1 1 5118AAE4
 P 9575 1575
 F 0 "U308" V 9350 1550 60  0000 C CNN
-F 1 "RGB_WS2811" V 9975 1550 60  0000 C CNN
-F 2 "TinyTiM_Lib:RGB_WS2811" H 9475 1975 60  0001 C CNN
+F 1 "RGB_WS2811B" V 9975 1550 60  0000 C CNN
+F 2 "TinyTiM_Lib:RGB_WS2811B" H 9475 1975 60  0001 C CNN
 F 3 "" H 9575 1575 60  0001 C CNN
 	1    9575 1575
@@
 	1150 2400 1150 2350
 Wire Wire Line
-	1400 1000 1400 750
-Wire Wire Line
 	9850 2350 9850 2200
 Wire Wire Line
@@
 Wire Wire Line
 	950  2350 9850 2350
-Connection ~ 1400 750
-Wire Wire Line
-	950  750  9450 750
 Connection ~ 4100 2350
 Connection ~ 6400 2350
@@
 Wire Wire Line
 	1600 2850 1600 2200
-Connection ~ 2550 750
-Wire Wire Line
-	2550 750  2550 1000
-Connection ~ 4850 750
-Wire Wire Line
-	4850 750  4850 1000
-Connection ~ 7150 750
-Wire Wire Line
-	7150 750  7150 1000
-Wire Wire Line
-	9450 750  9450 1000
-Wire Wire Line
-	8300 1000 8300 750
-Connection ~ 8300 750
-Wire Wire Line
-	6000 750  6000 1000
-Connection ~ 6000 750
-Wire Wire Line
-	3700 750  3700 1000
-Connection ~ 3700 750
 Wire Wire Line
 	8500 2850 8500 2200
