File: KiCad/rev2/Row_D.sch (KiCad schematic (older format))
At the start: 12 parts, among them U401 RGB_WS2811, U402 RGB_WS2811, U403 RGB_WS2811, U404 RGB_WS2811, U405 RGB_WS2811, U406 RGB_WS2811, U407 RGB_WS2811, U408 RGB_WS2811

Commit message: TinyTiM rev2 work in progress, schematic complete
Parts:
- U401, U402, U403, U404, U405, U406, U407, U408: value RGB_WS2811 -> RGB_WS2811B; footprint TinyTiM_Lib:RGB_WS2811 -> TinyTiM_Lib:RGB_WS2811B; symbol RGB_WS2811 -> RGB_WS2811B
Connections:
- net 5V: now also U401.1 (VDD), U402.1 (VDD), U403.1 (VDD), U404.1 (VDD), U405.1 (VDD), U406.1 (VDD), U407.1 (VDD), U408.1 (VDD); no longer U401.3 (VCC), U401.5 (VDD), U402.3 (VCC), U402.5 (VDD), U403.3 (VCC), U403.5 (VDD), U404.3 (VCC), U404.5 (VDD), U405.3 (VCC), U405.5 (VDD), U406.3 (VCC), U406.5 (VDD), U407.3 (VCC), U407.5 (VDD), U408.3 (VCC), U408.5 (VDD)
- net DI_D: now also U401.4 (DI); no longer U401.2 (DI)
- net DO_D: now also U408.2 (DO); no longer U408.1 (DO)
- net D_02: now also U401.2 (DO), U402.4 (DI); no longer U401.1 (DO), U402.2 (DI)
- net D_03: now also U402.2 (DO), U403.4 (DI); no longer U402.1 (DO), U403.2 (DI)
- net D_04: now also U403.2 (DO), U404.4 (DI); no longer U403.1 (DO), U404.2 (DI)
- net D_05: now also U404.2 (DO), U405.4 (DI); no longer U404.1 (DO), U405.2 (DI)
- net D_06: now also U405.2 (DO), U406.4 (DI); no longer U405.1 (DO), U406.2 (DI)
- net D_07: now also U406.2 (DO), U407.4 (DI); no longer U406.1 (DO), U407.2 (DI)
- net D_08: now also U407.2 (DO), U408.4 (DI); no longer U407.1 (DO), U408.2 (DI)
- net GND: now also U401.3 (VSS), U402.3 (VSS), U403.3 (VSS), U404.3 (VSS), U405.3 (VSS), U406.3 (VSS), U407.3 (VSS), U408.3 (VSS); no longer U401.6 (VSS), U402.6 (VSS), U403.6 (VSS), U404.6 (VSS), U405.6 (VSS), U406.6 (VSS), U407.6 (VSS), U408.6 (VSS)
- no-connect marks 10 -> 4
Changed lines of the file:
@@
 Text HLabel 950  900  0    60   Input ~ 0
 DI_D
-Text HLabel 950  750  0    60   Input ~ 0
+Text HLabel 950  2850 0    60   Input ~ 0
 5V
 $Comp
-L RGB_WS2811 U401
+L RGB_WS2811B U401
 U 1 1 5118ABBC
 P 1525 1575
 F 0 "U401" V 1300 1575 60  0000 C CNN
-F 1 "RGB_WS2811" V 1925 1550 60  0000 C CNN
-F 2 "TinyTiM_Lib:RGB_WS2811" H 1425 1975 60  0001 C CNN
+F 1 "RGB_WS2811B" V 1925 1550 60  0000 C CNN
+F 2 "TinyTiM_Lib:RGB_WS2811B" H 1425 1975 60  0001 C CNN
 F 3 "" H 1525 1575 60  0001 C CNN
 	1    1525 1575
 	1    0    0    -1
 $EndComp
-NoConn ~ 1400 2200
-NoConn ~ 2550 2200
-NoConn ~ 3700 2200
-NoConn ~ 4850 2200
-NoConn ~ 6000 2200
-NoConn ~ 7150 2200
 NoConn ~ 8300 2200
 NoConn ~ 9450 2200
-Text Label 950  750  0    60   ~ 0
-5V
 Text Label 950  2350 0    60   ~ 0
 GND
@@
 $EndComp
 $Comp
-L RGB_WS2811 U402
+L RGB_WS2811B U402
 U 1 1 5118AB0D
 P 2675 1575
 F 0 "U402" V 2450 1575 60  0000 C CNN
-F 1 "RGB_WS2811" V 3075 1550 60  0000 C CNN
-F 2 "TinyTiM_Lib:RGB_WS2811" H 2575 1975 60  0001 C CNN
+F 1 "RGB_WS2811B" V 3075 1550 60  0000 C CNN
+F 2 "TinyTiM_Lib:RGB_WS2811B" H 2575 1975 60  0001 C CNN
 F 3 "" H 2675 1575 60  0001 C CNN
 	1    2675 1575
@@
 $EndComp
 $Comp
-L RGB_WS2811 U403
+L RGB_WS2811B U403
 U 1 1 5118AB05
 P 3825 1575
 F 0 "U403" V 3600 1575 60  0000 C CNN
-F 1 "RGB_WS2811" V 4225 1550 60  0000 C CNN
-F 2 "TinyTiM_Lib:RGB_WS2811" H 3725 1975 60  0001 C CNN
+F 1 "RGB_WS2811B" V 4225 1550 60  0000 C CNN
+F 2 "TinyTiM_Lib:RGB_WS2811B" H 3725 1975 60  0001 C CNN
 F 3 "" H 3825 1575 60  0001 C CNN
 	1    3825 1575
@@
 $EndComp
 $Comp
-L RGB_WS2811 U404
+L RGB_WS2811B U404
 U 1 1 5118AB92
 P 4975 1575
 F 0 "U404" V 4750 1550 60  0000 C CNN
-F 1 "RGB_WS2811" V 5375 1550 60  0000 C CNN
-F 2 "TinyTiM_Lib:RGB_WS2811" H 4875 1975 60  0001 C CNN
+F 1 "RGB_WS2811B" V 5375 1550 60  0000 C CNN
+F 2 "TinyTiM_Lib:RGB_WS2811B" H 4875 1975 60  0001 C CNN
 F 3 "" H 4975 1575 60  0001 C CNN
 	1    4975 1575
@@
 $EndComp
 $Comp
-L RGB_WS2811 U405
+L RGB_WS2811B U405
 U 1 1 5118AAF9
 P 6125 1575
 F 0 "U405" V 5900 1550 60  0000 C CNN
-F 1 "RGB_WS2811" V 6525 1525 60  0000 C CNN
-F 2 "TinyTiM_Lib:RGB_WS2811" H 6025 1975 60  0001 C CNN
+F 1 "RGB_WS2811B" V 6525 1525 60  0000 C CNN
+F 2 "TinyTiM_Lib:RGB_WS2811B" H 6025 1975 60  0001 C CNN
 F 3 "" H 6125 1575 60  0001 C CNN
 	1    6125 1575
@@
 $EndComp
 $Comp
-L RGB_WS2811 U406
+L RGB_WS2811B U406
 U 1 1 51168947
 P 7275 1575
 F 0 "U406" V 7050 1550 60  0000 C CNN
-F 1 "RGB_WS2811" V 7675 1550 60  0000 C CNN
-F 2 "TinyTiM_Lib:RGB_WS2811" H 7175 1975 60  0001 C CNN
+F 1 "RGB_WS2811B" V 7675 1550 60  0000 C CNN
+F 2 "TinyTiM_Lib:RGB_WS2811B" H 7175 1975 60  0001 C CNN
 F 3 "" H 7275 1575 60  0001 C CNN
 	1    7275 1575
@@
 $EndComp
 $Comp
-L RGB_WS2811 U407
+L RGB_WS2811B U407
 U 1 1 5118AAED
 P 8425 1575
 F 0 "U407" V 8200 1550 60  0000 C CNN
-F 1 "RGB_WS2811" V 8825 1550 60  0000 C CNN
-F 2 "TinyTiM_Lib:RGB_WS2811" H 8325 1975 60  0001 C CNN
+F 1 "RGB_WS2811B" V 8825 1550 60  0000 C CNN
+F 2 "TinyTiM_Lib:RGB_WS2811B" H 8325 1975 60  0001 C CNN
 F 3 "" H 8425 1575 60  0001 C CNN
 	1    8425 1575
@@
 $EndComp
 $Comp
-L RGB_WS2811 U408
+L RGB_WS2811B U408
 U 1 1 5118AAE7
 P 9575 1575
 F 0 "U408" V 9350 1550 60  0000 C CNN
-F 1 "RGB_WS2811" V 9975 1550 60  0000 C CNN
-F 2 "TinyTiM_Lib:RGB_WS2811" H 9475 1975 60  0001 C CNN
+F 1 "RGB_WS2811B" V 9975 1550 60  0000 C CNN
+F 2 "TinyTiM_Lib:RGB_WS2811B" H 9475 1975 60  0001 C CNN
 F 3 "" H 9575 1575 60  0001 C CNN
 	1    9575 1575
@@
 	1150 2400 1150 2350
 Wire Wire Line
-	1400 1000 1400 750
-Wire Wire Line
 	9850 2350 9850 2200
 Wire Wire Line
@@
 Wire Wire Line
 	950  2350 9850 2350
-Connection ~ 1400 750
-Wire Wire Line
-	950  750  9450 750
 Connection ~ 4100 2350
 Connection ~ 6400 2350
@@
 Wire Wire Line
 	1600 2850 1600 2200
-Connection ~ 2550 750
-Wire Wire Line
-	2550 750  2550 1000
-Connection ~ 4850 750
-Wire Wire Line
-	4850 750  4850 1000
-Connection ~ 7150 750
-Wire Wire Line
-	7150 750  7150 1000
-Wire Wire Line
-	9450 750  9450 1000
-Wire Wire Line
-	8300 1000 8300 750
-Connection ~ 8300 750
-Wire Wire Line
-	6000 750  6000 1000
-Connection ~ 6000 750
-Wire Wire Line
-	3700 750  3700 1000
-Connection ~ 3700 750
 Wire Wire Line
 	8500 2850 8500 2200
