File: KiCad/rev2/Row_E.sch (KiCad schematic (older format))
At the start: 12 parts, among them U501 RGB_WS2811, U502 RGB_WS2811, U503 RGB_WS2811, U504 RGB_WS2811, U505 RGB_WS2811, U506 RGB_WS2811, U507 RGB_WS2811, U508 RGB_WS2811

Commit message: TinyTiM rev2 work in progress, schematic complete
Parts:
- U501, U502, U503, U504, U505, U506, U507, U508: value RGB_WS2811 -> RGB_WS2811B; footprint TinyTiM_Lib:RGB_WS2811 -> TinyTiM_Lib:RGB_WS2811B; symbol RGB_WS2811 -> RGB_WS2811B
Connections:
- net 5V: now also U501.1 (VDD), U502.1 (VDD), U503.1 (VDD), U504.1 (VDD), U505.1 (VDD), U506.1 (VDD), U507.1 (VDD), U508.1 (VDD); no longer U501.3 (VCC), U501.5 (VDD), U502.3 (VCC), U502.5 (VDD), U503.3 (VCC), U503.5 (VDD), U504.3 (VCC), U504.5 (VDD), U505.3 (VCC), U505.5 (VDD), U506.3 (VCC), U506.5 (VDD), U507.3 (VCC), U507.5 (VDD), U508.3 (VCC), U508.5 (VDD)
- net DI_E: now also U501.4 (DI); no longer U501.2 (DI)
- net DO_E: now also U508.2 (DO); no longer U508.1 (DO)
- net E_02: now also U501.2 (DO), U502.4 (DI); no longer U501.1 (DO), U502.2 (DI)
- net E_03: now also U502.2 (DO), U503.4 (DI); no longer U502.1 (DO), U503.2 (DI)
- net E_04: now also U503.2 (DO), U504.4 (DI); no longer U503.1 (DO), U504.2 (DI)
- net E_05: now also U504.2 (DO), U505.4 (DI); no longer U504.1 (DO), U505.2 (DI)
- net E_06: now also U505.2 (DO), U506.4 (DI); no longer U505.1 (DO), U506.2 (DI)
- net E_07: now also U506.2 (DO), U507.4 (DI); no longer U506.1 (DO), U507.2 (DI)
- net E_08: now also U507.2 (DO), U508.4 (DI); no longer U507.1 (DO), U508.2 (DI)
- net GND: now also U501.3 (VSS), U502.3 (VSS), U503.3 (VSS), U504.3 (VSS), U505.3 (VSS), U506.3 (VSS), U507.3 (VSS), U508.3 (VSS); no longer U501.6 (VSS), U502.6 (VSS), U503.6 (VSS), U504.6 (VSS), U505.6 (VSS), U506.6 (VSS), U507.6 (VSS), U508.6 (VSS)
- no-connect marks 10 -> 2
Changed lines of the file:
@@
 Text HLabel 950  900  0    60   Input ~ 0
 DI_E
-Text HLabel 950  750  0    60   Input ~ 0
-5V
-$Comp
-L RGB_WS2811 U501
+$Comp
+L RGB_WS2811B U501
 U 1 1 5118ABB9
 P 1525 1575
 F 0 "U501" V 1300 1575 60  0000 C CNN
-F 1 "RGB_WS2811" V 1925 1550 60  0000 C CNN
-F 2 "TinyTiM_Lib:RGB_WS2811" H 1425 1975 60  0001 C CNN
+F 1 "RGB_WS2811B" V 1925 1550 60  0000 C CNN
+F 2 "TinyTiM_Lib:RGB_WS2811B" H 1425 1975 60  0001 C CNN
 F 3 "" H 1525 1575 60  0001 C CNN
 	1    1525 1575
 	1    0    0    -1
 $EndComp
-NoConn ~ 1400 2200
-NoConn ~ 2550 2200
-NoConn ~ 3700 2200
-NoConn ~ 4850 2200
-NoConn ~ 6000 2200
-NoConn ~ 7150 2200
-NoConn ~ 8300 2200
-NoConn ~ 9450 2200
-Text Label 950  750  0    60   ~ 0
-5V
 Text Label 950  2350 0    60   ~ 0
 GND
@@
 $EndComp
 $Comp
-L RGB_WS2811 U502
+L RGB_WS2811B U502
 U 1 1 5118AB0A
 P 2675 1575
 F 0 "U502" V 2450 1575 60  0000 C CNN
-F 1 "RGB_WS2811" V 3075 1550 60  0000 C CNN
-F 2 "TinyTiM_Lib:RGB_WS2811" H 2575 1975 60  0001 C CNN
+F 1 "RGB_WS2811B" V 3075 1550 60  0000 C CNN
+F 2 "TinyTiM_Lib:RGB_WS2811B" H 2575 1975 60  0001 C CNN
 F 3 "" H 2675 1575 60  0001 C CNN
 	1    2675 1575
@@
 $EndComp
 $Comp
-L RGB_WS2811 U503
+L RGB_WS2811B U503
 U 1 1 5116894A
 P 3825 1575
 F 0 "U503" V 3600 1575 60  0000 C CNN
-F 1 "RGB_WS2811" V 4225 1550 60  0000 C CNN
-F 2 "TinyTiM_Lib:RGB_WS2811" H 3725 1975 60  0001 C CNN
+F 1 "RGB_WS2811B" V 4225 1550 60  0000 C CNN
+F 2 "TinyTiM_Lib:RGB_WS2811B" H 3725 1975 60  0001 C CNN
 F 3 "" H 3825 1575 60  0001 C CNN
 	1    3825 1575
@@
 $EndComp
 $Comp
-L RGB_WS2811 U504
+L RGB_WS2811B U504
 U 1 1 51189833
 P 4975 1575
 F 0 "U504" V 4750 1550 60  0000 C CNN
-F 1 "RGB_WS2811" V 5375 1550 60  0000 C CNN
-F 2 "TinyTiM_Lib:RGB_WS2811" H 4875 1975 60  0001 C CNN
+F 1 "RGB_WS2811B" V 5375 1550 60  0000 C CNN
+F 2 "TinyTiM_Lib:RGB_WS2811B" H 4875 1975 60  0001 C CNN
 F 3 "" H 4975 1575 60  0001 C CNN
 	1    4975 1575
@@
 $EndComp
 $Comp
-L RGB_WS2811 U505
+L RGB_WS2811B U505
 U 1 1 51168948
 P 6125 1575
 F 0 "U505" V 5900 1550 60  0000 C CNN
-F 1 "RGB_WS2811" V 6525 1525 60  0000 C CNN
-F 2 "TinyTiM_Lib:RGB_WS2811" H 6025 1975 60  0001 C CNN
+F 1 "RGB_WS2811B" V 6525 1525 60  0000 C CNN
+F 2 "TinyTiM_Lib:RGB_WS2811B" H 6025 1975 60  0001 C CNN
 F 3 "" H 6125 1575 60  0001 C CNN
 	1    6125 1575
@@
 $EndComp
 $Comp
-L RGB_WS2811 U506
+L RGB_WS2811B U506
 U 1 1 5118AAF7
 P 7275 1575
 F 0 "U506" V 7050 1550 60  0000 C CNN
-F 1 "RGB_WS2811" V 7675 1550 60  0000 C CNN
-F 2 "TinyTiM_Lib:RGB_WS2811" H 7175 1975 60  0001 C CNN
+F 1 "RGB_WS2811B" V 7675 1550 60  0000 C CNN
+F 2 "TinyTiM_Lib:RGB_WS2811B" H 7175 1975 60  0001 C CNN
 F 3 "" H 7275 1575 60  0001 C CNN
 	1    7275 1575
@@
 $EndComp
 $Comp
-L RGB_WS2811 U507
+L RGB_WS2811B U507
 U 1 1 5118AAEC
 P 8425 1575
 F 0 "U507" V 8200 1550 60  0000 C CNN
-F 1 "RGB_WS2811" V 8825 1550 60  0000 C CNN
-F 2 "TinyTiM_Lib:RGB_WS2811" H 8325 1975 60  0001 C CNN
+F 1 "RGB_WS2811B" V 8825 1550 60  0000 C CNN
+F 2 "TinyTiM_Lib:RGB_WS2811B" H 8325 1975 60  0001 C CNN
 F 3 "" H 8425 1575 60  0001 C CNN
 	1    8425 1575
@@
 $EndComp
 $Comp
-L RGB_WS2811 U508
+L RGB_WS2811B U508
 U 1 1 5118AAE9
 P 9575 1575
 F 0 "U508" V 9350 1550 60  0000 C CNN
-F 1 "RGB_WS2811" V 9975 1550 60  0000 C CNN
-F 2 "TinyTiM_Lib:RGB_WS2811" H 9475 1975 60  0001 C CNN
+F 1 "RGB_WS2811B" V 9975 1550 60  0000 C CNN
+F 2 "TinyTiM_Lib:RGB_WS2811B" H 9475 1975 60  0001 C CNN
 F 3 "" H 9575 1575 60  0001 C CNN
 	1    9575 1575
@@
 	1150 2400 1150 2350
 Wire Wire Line
-	1400 1000 1400 750
-Wire Wire Line
 	9850 2350 9850 2200
 Wire Wire Line
@@
 Wire Wire Line
 	950  2350 9850 2350
-Connection ~ 1400 750
-Wire Wire Line
-	950  750  9450 750
 Connection ~ 4100 2350
 Connection ~ 6400 2350
@@
 Wire Wire Line
 	1600 2850 1600 2200
-Connection ~ 2550 750
-Wire Wire Line
-	2550 750  2550 1000
-Connection ~ 4850 750
-Wire Wire Line
-	4850 750  4850 1000
-Connection ~ 7150 750
-Wire Wire Line
-	7150 750  7150 1000
-Wire Wire Line
-	9450 750  9450 1000
-Wire Wire Line
-	8300 1000 8300 750
-Connection ~ 8300 750
-Wire Wire Line
-	6000 750  6000 1000
-Connection ~ 6000 750
-Wire Wire Line
-	3700 750  3700 1000
-Connection ~ 3700 750
 Wire Wire Line
 	8500 2850 8500 2200
@@
 Wire Wire Line
 	1250 6550 1250 6350
+Text HLabel 950  2850 0    60   Input ~ 0
+5V
 $EndSCHEMATC
