File: KiCad/rev2/Row_F.sch (KiCad schematic (older format))
At the start: 10 parts, among them U601 RGB_WS2811, U602 RGB_WS2811, U603 RGB_WS2811, U604 RGB_WS2811, U605 RGB_WS2811, U606 RGB_WS2811, U607 RGB_WS2811, U608 RGB_WS2811

Commit message: TinyTiM rev2 work in progress, schematic complete
Parts:
- U601, U602, U603, U604, U605, U606, U607, U608: value RGB_WS2811 -> RGB_WS2811B; footprint TinyTiM_Lib:RGB_WS2811 -> TinyTiM_Lib:RGB_WS2811B; symbol RGB_WS2811 -> RGB_WS2811B
Connections:
- net 5V: now also U601.1 (VDD), U602.1 (VDD), U603.1 (VDD), U604.1 (VDD), U605.1 (VDD), U606.1 (VDD), U607.1 (VDD), U608.1 (VDD); no longer U601.3 (VCC), U601.5 (VDD), U602.3 (VCC), U602.5 (VDD), U603.3 (VCC), U603.5 (VDD), U604.3 (VCC), U604.5 (VDD), U605.3 (VCC), U605.5 (VDD), U606.3 (VCC), U606.5 (VDD), U607.3 (VCC), U607.5 (VDD), U608.3 (VCC), U608.5 (VDD)
- net DI_F: now also U601.4 (DI); no longer U601.2 (DI)
- net DO_F: now also U608.2 (DO); no longer U608.1 (DO)
- net F_02: now also U601.2 (DO), U602.4 (DI); no longer U601.1 (DO), U602.2 (DI)
- net F_03: now also U602.2 (DO), U603.4 (DI); no longer U602.1 (DO), U603.2 (DI)
- net F_04: now also U603.2 (DO), U604.4 (DI); no longer U603.1 (DO), U604.2 (DI)
- net F_05: now also U604.2 (DO), U605.4 (DI); no longer U604.1 (DO), U605.2 (DI)
- net F_06: now also U605.2 (DO), U606.4 (DI); no longer U605.1 (DO), U606.2 (DI)
- net F_07: now also U606.2 (DO), U607.4 (DI); no longer U606.1 (DO), U607.2 (DI)
- net F_08: now also U607.2 (DO), U608.4 (DI); no longer U607.1 (DO), U608.2 (DI)
- net GND: now also U601.3 (VSS), U602.3 (VSS), U603.3 (VSS), U604.3 (VSS), U605.3 (VSS), U606.3 (VSS), U607.3 (VSS), U608.3 (VSS); no longer U601.6 (VSS), U602.6 (VSS), U603.6 (VSS), U604.6 (VSS), U605.6 (VSS), U606.6 (VSS), U607.6 (VSS), U608.6 (VSS)
- no-connect marks 8 -> 0
Changed lines of the file:
@@
 Text HLabel 950  900  0    60   Input ~ 0
 DI_F
-Text HLabel 950  750  0    60   Input ~ 0
-5V
-$Comp
-L RGB_WS2811 U601
+$Comp
+L RGB_WS2811B U601
 U 1 1 5118ABB7
 P 1525 1575
 F 0 "U601" V 1300 1575 60  0000 C CNN
-F 1 "RGB_WS2811" V 1925 1550 60  0000 C CNN
-F 2 "TinyTiM_Lib:RGB_WS2811" H 1425 1975 60  0001 C CNN
+F 1 "RGB_WS2811B" V 1925 1550 60  0000 C CNN
+F 2 "TinyTiM_Lib:RGB_WS2811B" H 1425 1975 60  0001 C CNN
 F 3 "" H 1525 1575 60  0001 C CNN
 	1    1525 1575
 	1    0    0    -1
 $EndComp
-NoConn ~ 1400 2200
-NoConn ~ 2550 2200
-NoConn ~ 3700 2200
-NoConn ~ 4850 2200
-NoConn ~ 6000 2200
-NoConn ~ 7150 2200
-NoConn ~ 8300 2200
-NoConn ~ 9450 2200
-Text Label 950  750  0    60   ~ 0
-5V
 Text Label 950  2350 0    60   ~ 0
 GND
@@
 $EndComp
 $Comp
-L RGB_WS2811 U602
+L RGB_WS2811B U602
 U 1 1 5118AB0B
 P 2675 1575
 F 0 "U602" V 2450 1575 60  0000 C CNN
-F 1 "RGB_WS2811" V 3075 1550 60  0000 C CNN
-F 2 "TinyTiM_Lib:RGB_WS2811" H 2575 1975 60  0001 C CNN
+F 1 "RGB_WS2811B" V 3075 1550 60  0000 C CNN
+F 2 "TinyTiM_Lib:RGB_WS2811B" H 2575 1975 60  0001 C CNN
 F 3 "" H 2675 1575 60  0001 C CNN
 	1    2675 1575
@@
 $EndComp
 $Comp
-L RGB_WS2811 U603
+L RGB_WS2811B U603
 U 1 1 5118AB06
 P 3825 1575
 F 0 "U603" V 3600 1575 60  0000 C CNN
-F 1 "RGB_WS2811" V 4225 1550 60  0000 C CNN
-F 2 "TinyTiM_Lib:RGB_WS2811" H 3725 1975 60  0001 C CNN
+F 1 "RGB_WS2811B" V 4225 1550 60  0000 C CNN
+F 2 "TinyTiM_Lib:RGB_WS2811B" H 3725 1975 60  0001 C CNN
 F 3 "" H 3825 1575 60  0001 C CNN
 	1    3825 1575
@@
 $EndComp
 $Comp
-L RGB_WS2811 U604
+L RGB_WS2811B U604
 U 1 1 5118AB8C
 P 4975 1575
 F 0 "U604" V 4750 1550 60  0000 C CNN
-F 1 "RGB_WS2811" V 5375 1550 60  0000 C CNN
-F 2 "TinyTiM_Lib:RGB_WS2811" H 4875 1975 60  0001 C CNN
+F 1 "RGB_WS2811B" V 5375 1550 60  0000 C CNN
+F 2 "TinyTiM_Lib:RGB_WS2811B" H 4875 1975 60  0001 C CNN
 F 3 "" H 4975 1575 60  0001 C CNN
 	1    4975 1575
@@
 $EndComp
 $Comp
-L RGB_WS2811 U605
+L RGB_WS2811B U605
 U 1 1 5118AAFE
 P 6125 1575
 F 0 "U605" V 5900 1550 60  0000 C CNN
-F 1 "RGB_WS2811" V 6525 1525 60  0000 C CNN
-F 2 "TinyTiM_Lib:RGB_WS2811" H 6025 1975 60  0001 C CNN
+F 1 "RGB_WS2811B" V 6525 1525 60  0000 C CNN
+F 2 "TinyTiM_Lib:RGB_WS2811B" H 6025 1975 60  0001 C CNN
 F 3 "" H 6125 1575 60  0001 C CNN
 	1    6125 1575
@@
 $EndComp
 $Comp
-L RGB_WS2811 U606
+L RGB_WS2811B U606
 U 1 1 5118AAF6
 P 7275 1575
 F 0 "U606" V 7050 1550 60  0000 C CNN
-F 1 "RGB_WS2811" V 7675 1550 60  0000 C CNN
-F 2 "TinyTiM_Lib:RGB_WS2811" H 7175 1975 60  0001 C CNN
+F 1 "RGB_WS2811B" V 7675 1550 60  0000 C CNN
+F 2 "TinyTiM_Lib:RGB_WS2811B" H 7175 1975 60  0001 C CNN
 F 3 "" H 7275 1575 60  0001 C CNN
 	1    7275 1575
@@
 $EndComp
 $Comp
-L RGB_WS2811 U607
+L RGB_WS2811B U607
 U 1 1 51168946
 P 8425 1575
 F 0 "U607" V 8200 1550 60  0000 C CNN
-F 1 "RGB_WS2811" V 8825 1550 60  0000 C CNN
-F 2 "TinyTiM_Lib:RGB_WS2811" H 8325 1975 60  0001 C CNN
+F 1 "RGB_WS2811B" V 8825 1550 60  0000 C CNN
+F 2 "TinyTiM_Lib:RGB_WS2811B" H 8325 1975 60  0001 C CNN
 F 3 "" H 8425 1575 60  0001 C CNN
 	1    8425 1575
@@
 $EndComp
 $Comp
-L RGB_WS2811 U608
+L RGB_WS2811B U608
 U 1 1 51168945
 P 9575 1575
 F 0 "U608" V 9350 1550 60  0000 C CNN
-F 1 "RGB_WS2811" V 9975 1550 60  0000 C CNN
-F 2 "TinyTiM_Lib:RGB_WS2811" H 9475 1975 60  0001 C CNN
+F 1 "RGB_WS2811B" V 9975 1550 60  0000 C CNN
+F 2 "TinyTiM_Lib:RGB_WS2811B" H 9475 1975 60  0001 C CNN
 F 3 "" H 9575 1575 60  0001 C CNN
 	1    9575 1575
@@
 	1150 2400 1150 2350
 Wire Wire Line
-	1400 1000 1400 750
-Wire Wire Line
 	9850 2350 9850 2200
 Wire Wire Line
@@
 Wire Wire Line
 	950  2350 9850 2350
-Connection ~ 1400 750
-Wire Wire Line
-	950  750  9450 750
 Connection ~ 4100 2350
 Connection ~ 6400 2350
@@
 Wire Wire Line
 	1600 2850 1600 2200
-Connection ~ 2550 750
-Wire Wire Line
-	2550 750  2550 1000
-Connection ~ 4850 750
-Wire Wire Line
-	4850 750  4850 1000
-Connection ~ 7150 750
-Wire Wire Line
-	7150 750  7150 1000
-Wire Wire Line
-	9450 750  9450 1000
-Wire Wire Line
-	8300 1000 8300 750
-Connection ~ 8300 750
-Wire Wire Line
-	6000 750  6000 1000
-Connection ~ 6000 750
-Wire Wire Line
-	3700 750  3700 1000
-Connection ~ 3700 750
 Wire Wire Line
 	8500 2850 8500 2200
@@
 Wire Wire Line
 	1250 6550 1250 6350
+Text HLabel 950  2850 0    60   Input ~ 0
+5V
 $EndSCHEMATC
