File: KiCad/rev2/Row_G.sch (KiCad schematic (older format))
At the start: 10 parts, among them U701 RGB_WS2811, U702 RGB_WS2811, U703 RGB_WS2811, U704 RGB_WS2811, U705 RGB_WS2811, U706 RGB_WS2811, U707 RGB_WS2811, U708 RGB_WS2811

Commit message: TinyTiM rev2 work in progress, schematic complete
Parts:
- U701, U702, U703, U704, U705, U706, U707, U708: value RGB_WS2811 -> RGB_WS2811B; footprint TinyTiM_Lib:RGB_WS2811 -> TinyTiM_Lib:RGB_WS2811B; symbol RGB_WS2811 -> RGB_WS2811B
Connections:
- net 5V: now also U701.1 (VDD), U702.1 (VDD), U703.1 (VDD), U704.1 (VDD), U705.1 (VDD), U706.1 (VDD), U707.1 (VDD), U708.1 (VDD); no longer U701.3 (VCC), U701.5 (VDD), U702.3 (VCC), U702.5 (VDD), U703.3 (VCC), U703.5 (VDD), U704.3 (VCC), U704.5 (VDD), U705.3 (VCC), U705.5 (VDD), U706.3 (VCC), U706.5 (VDD), U707.3 (VCC), U707.5 (VDD), U708.3 (VCC), U708.5 (VDD)
- net DI_G: now also U701.4 (DI); no longer U701.2 (DI)
- net DO_G: now also U708.2 (DO); no longer U708.1 (DO)
- net GND: now also U701.3 (VSS), U702.3 (VSS), U703.3 (VSS), U704.3 (VSS), U705.3 (VSS), U706.3 (VSS), U707.3 (VSS), U708.3 (VSS); no longer U701.6 (VSS), U702.6 (VSS), U703.6 (VSS), U704.6 (VSS), U705.6 (VSS), U706.6 (VSS), U707.6 (VSS), U708.6 (VSS)
- net G_02: now also U701.2 (DO), U702.4 (DI); no longer U701.1 (DO), U702.2 (DI)
- net G_03: now also U702.2 (DO), U703.4 (DI); no longer U702.1 (DO), U703.2 (DI)
- net G_04: now also U703.2 (DO), U704.4 (DI); no longer U703.1 (DO), U704.2 (DI)
- net G_05: now also U704.2 (DO), U705.4 (DI); no longer U704.1 (DO), U705.2 (DI)
- net G_06: now also U705.2 (DO), U706.4 (DI); no longer U705.1 (DO), U706.2 (DI)
- net G_07: now also U706.2 (DO), U707.4 (DI); no longer U706.1 (DO), U707.2 (DI)
- net G_08: now also U707.2 (DO), U708.4 (DI); no longer U707.1 (DO), U708.2 (DI)
- no-connect marks 8 -> 0
Changed lines of the file:
@@
 Text HLabel 950  900  0    60   Input ~ 0
 DI_G
-Text HLabel 950  750  0    60   Input ~ 0
-5V
-$Comp
-L RGB_WS2811 U701
+$Comp
+L RGB_WS2811B U701
 U 1 1 5118ABB6
 P 1525 1575
 F 0 "U701" V 1300 1575 60  0000 C CNN
-F 1 "RGB_WS2811" V 1925 1550 60  0000 C CNN
-F 2 "TinyTiM_Lib:RGB_WS2811" H 1425 1975 60  0001 C CNN
+F 1 "RGB_WS2811B" V 1925 1550 60  0000 C CNN
+F 2 "TinyTiM_Lib:RGB_WS2811B" H 1425 1975 60  0001 C CNN
 F 3 "" H 1525 1575 60  0001 C CNN
 	1    1525 1575
 	1    0    0    -1
 $EndComp
-NoConn ~ 1400 2200
-NoConn ~ 2550 2200
-NoConn ~ 3700 2200
-NoConn ~ 4850 2200
-NoConn ~ 6000 2200
-NoConn ~ 7150 2200
-NoConn ~ 8300 2200
-NoConn ~ 9450 2200
-Text Label 950  750  0    60   ~ 0
-5V
 Text Label 950  2350 0    60   ~ 0
 GND
@@
 $EndComp
 $Comp
-L RGB_WS2811 U702
+L RGB_WS2811B U702
 U 1 1 5118AB07
 P 2675 1575
 F 0 "U702" V 2450 1575 60  0000 C CNN
-F 1 "RGB_WS2811" V 3075 1550 60  0000 C CNN
-F 2 "TinyTiM_Lib:RGB_WS2811" H 2575 1975 60  0001 C CNN
+F 1 "RGB_WS2811B" V 3075 1550 60  0000 C CNN
+F 2 "TinyTiM_Lib:RGB_WS2811B" H 2575 1975 60  0001 C CNN
 F 3 "" H 2675 1575 60  0001 C CNN
 	1    2675 1575
@@
 $EndComp
 $Comp
-L RGB_WS2811 U703
+L RGB_WS2811B U703
 U 1 1 5118AB04
 P 3825 1575
 F 0 "U703" V 3600 1575 60  0000 C CNN
-F 1 "RGB_WS2811" V 4225 1550 60  0000 C CNN
-F 2 "TinyTiM_Lib:RGB_WS2811" H 3725 1975 60  0001 C CNN
+F 1 "RGB_WS2811B" V 4225 1550 60  0000 C CNN
+F 2 "TinyTiM_Lib:RGB_WS2811B" H 3725 1975 60  0001 C CNN
 F 3 "" H 3825 1575 60  0001 C CNN
 	1    3825 1575
@@
 $EndComp
 $Comp
-L RGB_WS2811 U704
+L RGB_WS2811B U704
 U 1 1 5118AB8E
 P 4975 1575
 F 0 "U704" V 4750 1550 60  0000 C CNN
-F 1 "RGB_WS2811" V 5375 1550 60  0000 C CNN
-F 2 "TinyTiM_Lib:RGB_WS2811" H 4875 1975 60  0001 C CNN
+F 1 "RGB_WS2811B" V 5375 1550 60  0000 C CNN
+F 2 "TinyTiM_Lib:RGB_WS2811B" H 4875 1975 60  0001 C CNN
 F 3 "" H 4975 1575 60  0001 C CNN
 	1    4975 1575
@@
 $EndComp
 $Comp
-L RGB_WS2811 U705
+L RGB_WS2811B U705
 U 1 1 5118AAFD
 P 6125 1575
 F 0 "U705" V 5900 1550 60  0000 C CNN
-F 1 "RGB_WS2811" V 6525 1525 60  0000 C CNN
-F 2 "TinyTiM_Lib:RGB_WS2811" H 6025 1975 60  0001 C CNN
+F 1 "RGB_WS2811B" V 6525 1525 60  0000 C CNN
+F 2 "TinyTiM_Lib:RGB_WS2811B" H 6025 1975 60  0001 C CNN
 F 3 "" H 6125 1575 60  0001 C CNN
 	1    6125 1575
@@
 $EndComp
 $Comp
-L RGB_WS2811 U706
+L RGB_WS2811B U706
 U 1 1 5118AAF4
 P 7275 1575
 F 0 "U706" V 7050 1550 60  0000 C CNN
-F 1 "RGB_WS2811" V 7675 1550 60  0000 C CNN
-F 2 "TinyTiM_Lib:RGB_WS2811" H 7175 1975 60  0001 C CNN
+F 1 "RGB_WS2811B" V 7675 1550 60  0000 C CNN
+F 2 "TinyTiM_Lib:RGB_WS2811B" H 7175 1975 60  0001 C CNN
 F 3 "" H 7275 1575 60  0001 C CNN
 	1    7275 1575
@@
 $EndComp
 $Comp
-L RGB_WS2811 U707
+L RGB_WS2811B U707
 U 1 1 5118AAEF
 P 8425 1575
 F 0 "U707" V 8200 1550 60  0000 C CNN
-F 1 "RGB_WS2811" V 8825 1550 60  0000 C CNN
-F 2 "TinyTiM_Lib:RGB_WS2811" H 8325 1975 60  0001 C CNN
+F 1 "RGB_WS2811B" V 8825 1550 60  0000 C CNN
+F 2 "TinyTiM_Lib:RGB_WS2811B" H 8325 1975 60  0001 C CNN
 F 3 "" H 8425 1575 60  0001 C CNN
 	1    8425 1575
-	1    0    0    -1
-$EndComp
-$Comp
-L RGB_WS2811 U708
-U 1 1 5118AAE8
-P 9575 1575
-F 0 "U708" V 9350 1550 60  0000 C CNN
-F 1 "RGB_WS2811" V 9975 1550 60  0000 C CNN
-F 2 "TinyTiM_Lib:RGB_WS2811" H 9475 1975 60  0001 C CNN
-F 3 "" H 9575 1575 60  0001 C CNN
-	1    9575 1575
 	1    0    0    -1
 $EndComp
@@
 	1150 2400 1150 2350
 Wire Wire Line
-	1400 1000 1400 750
-Wire Wire Line
 	9850 2350 9850 2200
 Wire Wire Line
@@
 Wire Wire Line
 	950  2350 9850 2350
-Connection ~ 1400 750
-Wire Wire Line
-	950  750  9450 750
 Connection ~ 4100 2350
 Connection ~ 6400 2350
@@
 Wire Wire Line
 	1600 2850 1600 2200
-Connection ~ 2550 750
-Wire Wire Line
-	2550 750  2550 1000
-Connection ~ 4850 750
-Wire Wire Line
-	4850 750  4850 1000
-Connection ~ 7150 750
-Wire Wire Line
-	7150 750  7150 1000
-Wire Wire Line
-	9450 750  9450 1000
-Wire Wire Line
-	8300 1000 8300 750
-Connection ~ 8300 750
-Wire Wire Line
-	6000 750  6000 1000
-Connection ~ 6000 750
-Wire Wire Line
-	3700 750  3700 1000
-Connection ~ 3700 750
 Wire Wire Line
 	8500 2850 8500 2200
@@
 Wire Wire Line
 	1250 6550 1250 6350
+$Comp
+L RGB_WS2811B U708
+U 1 1 5118AAE8
+P 9575 1575
+F 0 "U708" V 9350 1550 60  0000 C CNN
+F 1 "RGB_WS2811B" V 9975 1550 60  0000 C CNN
+F 2 "TinyTiM_Lib:RGB_WS2811B" H 9475 1975 60  0001 C CNN
+F 3 "" H 9575 1575 60  0001 C CNN
+	1    9575 1575
+	1    0    0    -1
+$EndComp
+Text HLabel 950  2850 0    60   Input ~ 0
+5V
 $EndSCHEMATC
