File: KiCad/rev2/Row_H.sch (KiCad schematic (older format))
At the start: 14 parts, among them U801 RGB_WS2811, U802 RGB_WS2811, U803 RGB_WS2811, U804 RGB_WS2811, U805 RGB_WS2811, U806 RGB_WS2811, U807 RGB_WS2811, U808 RGB_WS2811

Commit message: TinyTiM rev2 work in progress, schematic complete
Parts:
- U801, U802, U803, U804, U805, U806, U807, U808: value RGB_WS2811 -> RGB_WS2811B; footprint TinyTiM_Lib:RGB_WS2811 -> TinyTiM_Lib:RGB_WS2811B; symbol RGB_WS2811 -> RGB_WS2811B
Connections:
- net 5V: now also U801.1 (VDD), U802.1 (VDD), U803.1 (VDD), U804.1 (VDD), U805.1 (VDD), U806.1 (VDD), U807.1 (VDD), U808.1 (VDD); no longer U801.3 (VCC), U801.5 (VDD), U802.3 (VCC), U802.5 (VDD), U803.3 (VCC), U803.5 (VDD), U804.3 (VCC), U804.5 (VDD), U805.3 (VCC), U805.5 (VDD), U806.3 (VCC), U806.5 (VDD), U807.3 (VCC), U807.5 (VDD), U808.3 (VCC), U808.5 (VDD)
- net DI_H: now also U801.4 (DI); no longer U801.2 (DI)
- net DO_H: now also U808.2 (DO); no longer U808.1 (DO)
- net GND: now also U801.3 (VSS), U802.3 (VSS), U803.3 (VSS), U804.3 (VSS), U805.3 (VSS), U806.3 (VSS), U807.3 (VSS), U808.3 (VSS); no longer U801.6 (VSS), U802.6 (VSS), U803.6 (VSS), U804.6 (VSS), U805.6 (VSS), U806.6 (VSS), U807.6 (VSS), U808.6 (VSS)
- net H_02: now also U801.2 (DO), U802.4 (DI); no longer U801.1 (DO), U802.2 (DI)
- net H_03: now also U802.2 (DO), U803.4 (DI); no longer U802.1 (DO), U803.2 (DI)
- net H_04: now also U803.2 (DO), U804.4 (DI); no longer U803.1 (DO), U804.2 (DI)
- net H_05: now also U804.2 (DO), U805.4 (DI); no longer U804.1 (DO), U805.2 (DI)
- net H_06: now also U805.2 (DO), U806.4 (DI); no longer U805.1 (DO), U806.2 (DI)
- net H_07: now also U806.2 (DO), U807.4 (DI); no longer U806.1 (DO), U807.2 (DI)
- net H_08: now also U807.2 (DO), U808.4 (DI); no longer U807.1 (DO), U808.2 (DI)
- no-connect marks 12 -> 4
Changed lines of the file:
@@
 Text HLabel 950  900  0    60   Input ~ 0
 DI_H
-Text HLabel 950  750  0    60   Input ~ 0
-5V
-$Comp
-L RGB_WS2811 U801
+$Comp
+L RGB_WS2811B U801
 U 1 1 5118ABBB
 P 1525 1575
 F 0 "U801" V 1300 1575 60  0000 C CNN
-F 1 "RGB_WS2811" V 1925 1550 60  0000 C CNN
-F 2 "TinyTiM_Lib:RGB_WS2811" H 1425 1975 60  0001 C CNN
+F 1 "RGB_WS2811B" V 1925 1550 60  0000 C CNN
+F 2 "TinyTiM_Lib:RGB_WS2811B" H 1425 1975 60  0001 C CNN
 F 3 "" H 1525 1575 60  0001 C CNN
 	1    1525 1575
 	1    0    0    -1
 $EndComp
-NoConn ~ 1400 2200
-NoConn ~ 2550 2200
-NoConn ~ 3700 2200
-NoConn ~ 4850 2200
-NoConn ~ 6000 2200
-NoConn ~ 7150 2200
-NoConn ~ 8300 2200
-NoConn ~ 9450 2200
-Text Label 950  750  0    60   ~ 0
-5V
 Text Label 950  2350 0    60   ~ 0
 GND
@@
 $EndComp
 $Comp
-L RGB_WS2811 U802
+L RGB_WS2811B U802
 U 1 1 5118AB09
 P 2675 1575
 F 0 "U802" V 2450 1575 60  0000 C CNN
-F 1 "RGB_WS2811" V 3075 1550 60  0000 C CNN
-F 2 "TinyTiM_Lib:RGB_WS2811" H 2575 1975 60  0001 C CNN
+F 1 "RGB_WS2811B" V 3075 1550 60  0000 C CNN
+F 2 "TinyTiM_Lib:RGB_WS2811B" H 2575 1975 60  0001 C CNN
 F 3 "" H 2675 1575 60  0001 C CNN
 	1    2675 1575
@@
 $EndComp
 $Comp
-L RGB_WS2811 U803
+L RGB_WS2811B U803
 U 1 1 5118AB03
 P 3825 1575
 F 0 "U803" V 3600 1575 60  0000 C CNN
-F 1 "RGB_WS2811" V 4225 1550 60  0000 C CNN
-F 2 "TinyTiM_Lib:RGB_WS2811" H 3725 1975 60  0001 C CNN
+F 1 "RGB_WS2811B" V 4225 1550 60  0000 C CNN
+F 2 "TinyTiM_Lib:RGB_WS2811B" H 3725 1975 60  0001 C CNN
 F 3 "" H 3825 1575 60  0001 C CNN
 	1    3825 1575
@@
 $EndComp
 $Comp
-L RGB_WS2811 U804
+L RGB_WS2811B U804
 U 1 1 5118AB8F
 P 4975 1575
 F 0 "U804" V 4750 1550 60  0000 C CNN
-F 1 "RGB_WS2811" V 5375 1550 60  0000 C CNN
-F 2 "TinyTiM_Lib:RGB_WS2811" H 4875 1975 60  0001 C CNN
+F 1 "RGB_WS2811B" V 5375 1550 60  0000 C CNN
+F 2 "TinyTiM_Lib:RGB_WS2811B" H 4875 1975 60  0001 C CNN
 F 3 "" H 4975 1575 60  0001 C CNN
 	1    4975 1575
@@
 $EndComp
 $Comp
-L RGB_WS2811 U805
+L RGB_WS2811B U805
 U 1 1 5118AAFF
 P 6125 1575
 F 0 "U805" V 5900 1550 60  0000 C CNN
-F 1 "RGB_WS2811" V 6525 1525 60  0000 C CNN
-F 2 "TinyTiM_Lib:RGB_WS2811" H 6025 1975 60  0001 C CNN
+F 1 "RGB_WS2811B" V 6525 1525 60  0000 C CNN
+F 2 "TinyTiM_Lib:RGB_WS2811B" H 6025 1975 60  0001 C CNN
 F 3 "" H 6125 1575 60  0001 C CNN
 	1    6125 1575
@@
 $EndComp
 $Comp
-L RGB_WS2811 U806
+L RGB_WS2811B U806
 U 1 1 5118AAF8
 P 7275 1575
 F 0 "U806" V 7050 1550 60  0000 C CNN
-F 1 "RGB_WS2811" V 7675 1550 60  0000 C CNN
-F 2 "TinyTiM_Lib:RGB_WS2811" H 7175 1975 60  0001 C CNN
+F 1 "RGB_WS2811B" V 7675 1550 60  0000 C CNN
+F 2 "TinyTiM_Lib:RGB_WS2811B" H 7175 1975 60  0001 C CNN
 F 3 "" H 7275 1575 60  0001 C CNN
 	1    7275 1575
@@
 $EndComp
 $Comp
-L RGB_WS2811 U807
+L RGB_WS2811B U807
 U 1 1 5118AAF1
 P 8425 1575
 F 0 "U807" V 8200 1550 60  0000 C CNN
-F 1 "RGB_WS2811" V 8825 1550 60  0000 C CNN
-F 2 "TinyTiM_Lib:RGB_WS2811" H 8325 1975 60  0001 C CNN
+F 1 "RGB_WS2811B" V 8825 1550 60  0000 C CNN
+F 2 "TinyTiM_Lib:RGB_WS2811B" H 8325 1975 60  0001 C CNN
 F 3 "" H 8425 1575 60  0001 C CNN
 	1    8425 1575
@@
 $EndComp
 $Comp
-L RGB_WS2811 U808
+L RGB_WS2811B U808
 U 1 1 5118AAE6
 P 9575 1575
 F 0 "U808" V 9350 1550 60  0000 C CNN
-F 1 "RGB_WS2811" V 9975 1550 60  0000 C CNN
-F 2 "TinyTiM_Lib:RGB_WS2811" H 9475 1975 60  0001 C CNN
+F 1 "RGB_WS2811B" V 9975 1550 60  0000 C CNN
+F 2 "TinyTiM_Lib:RGB_WS2811B" H 9475 1975 60  0001 C CNN
 F 3 "" H 9575 1575 60  0001 C CNN
 	1    9575 1575
@@
 	1150 2400 1150 2350
 Wire Wire Line
-	1400 1000 1400 750
-Wire Wire Line
 	9850 2350 9850 2200
 Wire Wire Line
@@
 Wire Wire Line
 	950  2350 9850 2350
-Connection ~ 1400 750
-Wire Wire Line
-	950  750  9450 750
 Connection ~ 4100 2350
 Connection ~ 6400 2350
@@
 Wire Wire Line
 	1600 2850 1600 2200
-Connection ~ 2550 750
-Wire Wire Line
-	2550 750  2550 1000
-Connection ~ 4850 750
-Wire Wire Line
-	4850 750  4850 1000
-Connection ~ 7150 750
-Wire Wire Line
-	7150 750  7150 1000
-Wire Wire Line
-	9450 750  9450 1000
-Wire Wire Line
-	8300 1000 8300 750
-Connection ~ 8300 750
-Wire Wire Line
-	6000 750  6000 1000
-Connection ~ 6000 750
-Wire Wire Line
-	3700 750  3700 1000
-Connection ~ 3700 750
 Wire Wire Line
 	8500 2850 8500 2200
@@
 NoConn ~ 5700 6800
 NoConn ~ 5900 6800
+Text HLabel 950  2850 0    60   Input ~ 0
+5V
 $EndSCHEMATC
