File: KiCad/rev2/TinyTiM.sch (KiCad schematic (older format))
At the start: 15 parts, among them P1 PWR_W, P125 G>H, P126 F>G, P127 E>F, P128 D>E, P129 C>D, P130 B>C, P131 A>B, P2 PWR_E, P3 Data_In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

Commit message: TinyTiM rev2 work in progress, schematic complete
Parts:
- P5, P6: footprint Conn_x3_PTSM -> TinyTiM_Lib:Conn_x3_PTSM
Changed lines of the file:
@@
 01 31 04 0B 88 21 58 40 0C C1 02 62 08 16 10 43 B0 80 18 82 05 C4 10 2C 20 86 60 01 31 04 0B 88
 21 58 40 0C C1 02 62 08 16 10 43 B0 80 18 82 05 C4 10 2C 20 86 60 01 31 04 0B 88 21 58 40 0C C1
-02 62 7C 03 3D 79 5E 0E 30 13 47 E7 00 00 00 00 49 45 4E 44 AE 42 60 82 91
+02 62 7C 03 3D 79 5E 0E 30 13 47 E7 00 00 00 00 49 45 4E 44 AE 42 60 82 41
 EndData
 $EndBitmap
@@
 C1 ED 35 72 E0 F7 FB FF F1 1F FF F1 9F FF F9 9F C7 C7 C7 73 1A 9F 2B 70 38 1C FB F6 ED 3B 79 F2
 E4 23 8F 3C 52 B0 F1 D9 2E 76 F1 FF 03 17 ED 19 47 28 92 59 FB 00 00 00 00 49 45 4E 44 AE 42 60
-82 3D
+82 00
 EndData
 $EndBitmap
@@
 F 0 "P5" H 1350 3250 50  0000 C CNN
 F 1 "Data_In_Serial" H 1350 3650 50  0000 C CNN
-F 2 "Conn_x3_PTSM" H 1350 3400 60  0001 C CNN
+F 2 "TinyTiM_Lib:Conn_x3_PTSM" H 1350 3400 60  0001 C CNN
 F 3 "" H 1350 3400 60  0000 C CNN
 F 4 "CONN HEADER 50POS .100\" SGL GOLD" H 1350 3500 60  0001 L CNN "Field4"
@@
 F 0 "P6" H 5450 3250 50  0000 C CNN
 F 1 "Data_Out_Serial" H 5450 3650 50  0000 C CNN
-F 2 "Conn_x3_PTSM" H 5450 3400 60  0001 C CNN
+F 2 "TinyTiM_Lib:Conn_x3_PTSM" H 5450 3400 60  0001 C CNN
 F 3 "" H 5450 3400 60  0000 C CNN
 F 4 "CONN HEADER 50POS .100\" SGL GOLD" H 5450 3500 60  0001 L CNN "Field4"
