File: KiCad/uTiM/Row_E.sch (KiCad schematic (older format))
At the start: 12 parts, among them U501 APA102, U502 APA102, U503 APA102, U504 APA102, U505 APA102, U506 APA102, U507 APA102, U508 APA102

Commit message: microTiM aka uTiM work in progress
Parts:
- S501, S502: value CONN_1 -> MH
Connections:
- net CO_E renamed CI_F
- net DO_E renamed DI_F
Changed lines of the file:
@@
 P 5300 6650
 F 0 "S501" V 5380 6650 40  0000 L CNN
-F 1 "CONN_1" H 5300 6705 30  0001 C CNN
+F 1 "MH" H 5300 6705 30  0001 C CNN
 F 2 "TinyTiM_Libs:Screw_NPTH" H 5300 6805 30  0001 C CNN
 F 3 "" H 5300 6650 60  0001 C CNN
@@
 P 5500 6650
 F 0 "S502" V 5580 6650 40  0000 L CNN
-F 1 "CONN_1" H 5500 6705 30  0001 C CNN
+F 1 "MH" H 5500 6705 30  0001 C CNN
 F 2 "TinyTiM_Libs:Screw_NPTH" H 5500 6805 30  0001 C CNN
 F 3 "" H 5500 6650 60  0001 C CNN
@@
 DI_E
 Text HLabel 950  3100 0    60   Output ~ 12
-CO_E
+CI_F
 Text HLabel 950  2350 0    60   Input ~ 12
 GND
@@
 5V
 Text Label 1075 3100 0    60   ~ 0
-CO_E
+CI_F
 $Comp
 L GND #PWR07
@@
 	10950 3350 950  3350
 Text HLabel 950  3350 0    60   Output ~ 12
-DO_E
+DI_F
 Text HLabel 950  1400 0    60   Input ~ 12
 DI_E
@@
 	1300 1600 950  1600
 Text Label 1075 3350 0    60   ~ 0
-DO_E
+DI_F
 Text Label 1075 1600 0    60   ~ 0
 CI_E

Commit message: work in progress, microTIM using APA102
Parts:
- removed C501: 100n, TinyTiM_Libs:c_0805, symbol C2
- removed C517: 47u,8V, TinyTiM_Libs:c_2917, symbol C_POL_1
- removed S501, S502: MH, TinyTiM_Libs:Screw_NPTH, symbol LOGO_1
Other:
- note removed: "Mounting Screws"
Changed lines of the file:
@@
 Comment4 ""
 $EndDescr
-$Comp
-L C2 C501
-U 1 1 5118AB5A
-P 1800 2600
-F 0 "C501" H 1825 2700 40  0000 L CNB
-F 1 "100n" H 1825 2500 40  0000 L CNN
-F 2 "TinyTiM_Libs:c_0805" H 1800 2600 50  0001 C CNN
-F 3 "" H 1800 2600 60  0001 C CNN
-F 4 "CAP CER 0.1UF 25V 10% X7R 0805" H 1800 2800 60  0001 L CNN "Field4"
-F 5 "100nF, 25V" H 1800 2900 60  0001 L CNN "Field5"
-F 6 "Surface Mount, MLCC" H 1800 3000 60  0001 L CNN "Field6"
-F 7 "Kemet" H 1800 3100 60  0001 L CNN "Field7"
-F 8 "C0805C104K3RACTU" H 1800 3200 60  0001 L CNN "Field8"
-F 9 "Digikey" H 1800 3300 60  0001 L CNN "Field9"
-F 10 "399-1168-1-ND" H 1800 3400 60  0001 L CNN "Field10"
-F 11 "http://www.digikey.com/product-detail/en/C0805C104K3RACTU/399-1168-1-ND/411443" H 1800 3500 60  0001 L CNN "Field11"
-	1    1800 2600
-	1    0    0    -1
-$EndComp
-$Comp
-L LOGO_1 S501
-U 1 1 51189825
-P 5300 6650
-F 0 "S501" V 5380 6650 40  0000 L CNN
-F 1 "MH" H 5300 6705 30  0001 C CNN
-F 2 "TinyTiM_Libs:Screw_NPTH" H 5300 6805 30  0001 C CNN
-F 3 "" H 5300 6650 60  0001 C CNN
-	1    5300 6650
-	0    -1   -1   0
-$EndComp
-$Comp
-L LOGO_1 S502
-U 1 1 51189824
-P 5500 6650
-F 0 "S502" V 5580 6650 40  0000 L CNN
-F 1 "MH" H 5500 6705 30  0001 C CNN
-F 2 "TinyTiM_Libs:Screw_NPTH" H 5500 6805 30  0001 C CNN
-F 3 "" H 5500 6650 60  0001 C CNN
-	1    5500 6650
-	0    -1   -1   0
-$EndComp
-Text Notes 5200 7000 0    60   ~ 0
-Mounting Screws
-Text Label 1250 6350 0    60   ~ 0
-5V
-Text Label 1250 7200 0    60   ~ 0
-GND
-$Comp
-L C_POL_1 C517
-U 1 1 51189821
-P 1250 6750
-F 0 "C517" H 1375 6725 40  0000 L CNB
-F 1 "47u,8V" H 1375 6625 40  0000 L CNN
-F 2 "TinyTiM_Libs:c_2917" H 1250 6700 50  0001 C CNN
-F 3 "" H 1250 6750 60  0001 C CNN
-F 4 "CAP ALUM 47UF 8V 20% SMD" H 1250 6950 60  0001 L CNN "Field4"
-F 5 "47u,8V" H 1250 7050 60  0001 L CNN "Field5"
-F 6 "2917 (7343 Metric)" H 1250 7150 60  0001 L CNN "Field6"
-F 7 "Panasonic Electronic Components" H 1250 7250 60  0001 L CNN "Field7"
-F 8 "EEF-CD0K470R" H 1250 7350 60  0001 L CNN "Field8"
-F 9 "Digikey" H 1250 7450 60  0001 L CNN "Field9"
-F 10 "PCE3606CT-ND" H 1250 7550 60  0001 L CNN "Field10"
-F 11 "http://www.digikey.com/product-detail/en/EEF-CD0K470R/PCE3606CT-ND/614442" H 1250 7650 60  0001 L CNN "Field11"
-	1    1250 6750
-	1    0    0    -1
-$EndComp
-Wire Wire Line
-	1250 7000 1250 7200
-Wire Wire Line
-	1250 6550 1250 6350
 Text Label 1075 1400 0    60   ~ 0
 DI_E
@@
 Wire Wire Line
 	1150 1800 1150 2400
-Connection ~ 1800 2850
-Wire Wire Line
-	1800 2850 1800 2800
 Wire Wire Line
 	950  3100 10800 3100
-Connection ~ 1800 2350
 Wire Wire Line
 	950  2350 9550 2350
@@
 	10800 3100 10800 1600
 Wire Wire Line
-	1800 2350 1800 2400
-Wire Wire Line
 	950  2850 10650 2850

Commit message: layout complete. Gerbers pending
Parts:
- renumbered U501 to U33, U502 to U34, U503 to U35, U504 to U36, U505 to U37, U506 to U38, U507 to U39, U508 to U40
Changed lines of the file:
@@
 GND
 $Comp
-L APA102 U501
+L APA102 U33
 U 1 1 56C24FAA
 P 1700 1600
-F 0 "U501" H 1700 1900 40  0000 C CNB
+F 0 "U33" H 1700 1900 40  0000 C CNB
 F 1 "APA102" H 1700 1275 40  0000 C CNN
 F 2 "TinyTiM_Libs:APA102" H 1600 2000 60  0001 C CNN
@@
 5V
 $Comp
-L APA102 U502
+L APA102 U34
 U 1 1 56C24FD5
 P 2900 1600
-F 0 "U502" H 2900 1900 40  0000 C CNB
+F 0 "U34" H 2900 1900 40  0000 C CNB
 F 1 "APA102" H 2900 1275 40  0000 C CNN
 F 2 "TinyTiM_Libs:APA102" H 2800 2000 60  0001 C CNN
@@
 $EndComp
 $Comp
-L APA102 U503
+L APA102 U35
 U 1 1 56C24FDD
 P 4100 1600
-F 0 "U503" H 4100 1900 40  0000 C CNB
+F 0 "U35" H 4100 1900 40  0000 C CNB
 F 1 "APA102" H 4100 1275 40  0000 C CNN
 F 2 "TinyTiM_Libs:APA102" H 4000 2000 60  0001 C CNN
@@
 $EndComp
 $Comp
-L APA102 U504
+L APA102 U36
 U 1 1 56C24FE5
 P 5300 1600
-F 0 "U504" H 5300 1900 40  0000 C CNB
+F 0 "U36" H 5300 1900 40  0000 C CNB
 F 1 "APA102" H 5300 1275 40  0000 C CNN
 F 2 "TinyTiM_Libs:APA102" H 5200 2000 60  0001 C CNN
@@
 $EndComp
 $Comp
-L APA102 U505
+L APA102 U37
 U 1 1 56C24FED
 P 6500 1600
-F 0 "U505" H 6500 1900 40  0000 C CNB
+F 0 "U37" H 6500 1900 40  0000 C CNB
 F 1 "APA102" H 6500 1275 40  0000 C CNN
 F 2 "TinyTiM_Libs:APA102" H 6400 2000 60  0001 C CNN
@@
 $EndComp
 $Comp
-L APA102 U506
+L APA102 U38
 U 1 1 56C24FF5
 P 7700 1600
-F 0 "U506" H 7700 1900 40  0000 C CNB
+F 0 "U38" H 7700 1900 40  0000 C CNB
 F 1 "APA102" H 7700 1275 40  0000 C CNN
 F 2 "TinyTiM_Libs:APA102" H 7600 2000 60  0001 C CNN
@@
 $EndComp
 $Comp
-L APA102 U507
+L APA102 U39
 U 1 1 56C24FFD
 P 8900 1600
-F 0 "U507" H 8900 1900 40  0000 C CNB
+F 0 "U39" H 8900 1900 40  0000 C CNB
 F 1 "APA102" H 8900 1275 40  0000 C CNN
 F 2 "TinyTiM_Libs:APA102" H 8800 2000 60  0001 C CNN
@@
 $EndComp
 $Comp
-L APA102 U508
+L APA102 U40
 U 1 1 56C25005
 P 10100 1600
-F 0 "U508" H 10100 1900 40  0000 C CNB
+F 0 "U40" H 10100 1900 40  0000 C CNB
 F 1 "APA102" H 10100 1275 40  0000 C CNN
 F 2 "TinyTiM_Libs:APA102" H 10000 2000 60  0001 C CNN
