File: KiCad/uTiM/Row_H.sch (KiCad schematic (older format))
At the start: 16 parts, among them U801 APA102, U802 APA102, U803 APA102, U804 APA102, U805 APA102, U806 APA102, U807 APA102, U808 APA102

Commit message: microTiM aka uTiM work in progress
Parts:
- S801: value CONN_1 -> 5V; footprint TinyTiM_Libs:Screw_SSide -> TinyTiM_Libs:PowerIn_stud; manf# (none) -> Value
- S802: value CONN_1 -> GND; footprint TinyTiM_Libs:Screw_SSide -> TinyTiM_Libs:PowerIn_stud; manf# (none) -> Value
- S803, S804: value CONN_1 -> MH
- S805: value CONN_1 -> DO_H; footprint TinyTiM_Libs:Screw_SSide -> TinyTiM_Libs:Contact_SMD
- S806: value CONN_1 -> CO_H; footprint TinyTiM_Libs:Screw_SSide -> TinyTiM_Libs:Contact_SMD
Changed lines of the file:
@@
 P 5100 6650
 F 0 "S801" V 5180 6650 40  0000 L CNN
-F 1 "CONN_1" H 5100 6705 30  0001 C CNN
-F 2 "TinyTiM_Libs:Screw_SSide" H 5100 6805 30  0001 C CNN
+F 1 "5V" H 5100 6705 30  0001 C CNN
+F 2 "TinyTiM_Libs:PowerIn_stud" H 5100 6805 30  0001 C CNN
 F 3 "" H 5100 6650 60  0001 C CNN
+F 4 "Value" H 5100 6650 60  0001 C CNN "manf#"
 	1    5100 6650
 	0    1    1    0
@@
 P 5400 6650
 F 0 "S802" V 5480 6650 40  0000 L CNN
-F 1 "CONN_1" H 5400 6705 30  0001 C CNN
-F 2 "TinyTiM_Libs:Screw_SSide" H 5400 6805 30  0001 C CNN
+F 1 "GND" H 5400 6705 30  0001 C CNN
+F 2 "TinyTiM_Libs:PowerIn_stud" H 5400 6805 30  0001 C CNN
 F 3 "" H 5400 6650 60  0001 C CNN
+F 4 "Value" H 5400 6650 60  0001 C CNN "manf#"
 	1    5400 6650
 	0    -1   -1   0
@@
 P 5700 6650
 F 0 "S803" V 5780 6650 40  0000 L CNN
-F 1 "CONN_1" H 5700 6705 30  0001 C CNN
+F 1 "MH" H 5700 6705 30  0001 C CNN
 F 2 "TinyTiM_Libs:Screw_NPTH" H 5700 6805 30  0001 C CNN
 F 3 "" H 5700 6650 60  0001 C CNN
@@
 P 5900 6650
 F 0 "S804" V 5980 6650 40  0000 L CNN
-F 1 "CONN_1" H 5900 6705 30  0001 C CNN
+F 1 "MH" H 5900 6705 30  0001 C CNN
 F 2 "TinyTiM_Libs:Screw_NPTH" H 5900 6805 30  0001 C CNN
 F 3 "" H 5900 6650 60  0001 C CNN
@@
 P 4500 6650
 F 0 "S806" V 4580 6650 40  0000 L CNN
-F 1 "CONN_1" H 4500 6705 30  0001 C CNN
-F 2 "TinyTiM_Libs:Screw_SSide" H 4500 6805 30  0001 C CNN
+F 1 "CO_H" H 4500 6705 30  0001 C CNN
+F 2 "TinyTiM_Libs:Contact_SMD" H 4500 6805 30  0001 C CNN
 F 3 "" H 4500 6650 60  0001 C CNN
 	1    4500 6650
@@
 P 4100 6650
 F 0 "S805" V 4180 6650 40  0000 L CNN
-F 1 "CONN_1" H 4100 6705 30  0001 C CNN
-F 2 "TinyTiM_Libs:Screw_SSide" H 4100 6805 30  0001 C CNN
+F 1 "DO_H" H 4100 6705 30  0001 C CNN
+F 2 "TinyTiM_Libs:Contact_SMD" H 4100 6805 30  0001 C CNN
 F 3 "" H 4100 6650 60  0001 C CNN
 	1    4100 6650

Commit message: work in progress, microTIM using APA102
Parts:
- removed S801: 5V, TinyTiM_Libs:PowerIn_stud, symbol CONN_1
- removed S802: GND, TinyTiM_Libs:PowerIn_stud, symbol CONN_1
- removed S803, S804: MH, TinyTiM_Libs:Screw_NPTH, symbol LOGO_1
- removed S805: DO_H, TinyTiM_Libs:Contact_SMD, symbol CONN_1
- removed S806: CO_H, TinyTiM_Libs:Contact_SMD, symbol CONN_1
Other:
- note removed: "Mounting Screws"
Changed lines of the file:
@@
 	1    0    0    -1
 $EndComp
-$Comp
-L CONN_1 S801
-U 1 1 5118AB78
-P 5100 6650
-F 0 "S801" V 5180 6650 40  0000 L CNN
-F 1 "5V" H 5100 6705 30  0001 C CNN
-F 2 "TinyTiM_Libs:PowerIn_stud" H 5100 6805 30  0001 C CNN
-F 3 "" H 5100 6650 60  0001 C CNN
-F 4 "Value" H 5100 6650 60  0001 C CNN "manf#"
-	1    5100 6650
-	0    1    1    0
-$EndComp
-$Comp
-L CONN_1 S802
-U 1 1 5118AB70
-P 5400 6650
-F 0 "S802" V 5480 6650 40  0000 L CNN
-F 1 "GND" H 5400 6705 30  0001 C CNN
-F 2 "TinyTiM_Libs:PowerIn_stud" H 5400 6805 30  0001 C CNN
-F 3 "" H 5400 6650 60  0001 C CNN
-F 4 "Value" H 5400 6650 60  0001 C CNN "manf#"
-	1    5400 6650
-	0    -1   -1   0
-$EndComp
-Text Notes 5200 7300 0    60   ~ 0
-Mounting Screws
 Text Label 1250 6350 0    60   ~ 0
 5V
@@
 Wire Wire Line
 	1250 6550 1250 6350
-$Comp
-L LOGO_1 S803
-U 1 1 5356BE2F
-P 5700 6650
-F 0 "S803" V 5780 6650 40  0000 L CNN
-F 1 "MH" H 5700 6705 30  0001 C CNN
-F 2 "TinyTiM_Libs:Screw_NPTH" H 5700 6805 30  0001 C CNN
-F 3 "" H 5700 6650 60  0001 C CNN
-	1    5700 6650
-	0    -1   -1   0
-$EndComp
-$Comp
-L LOGO_1 S804
-U 1 1 5356BE35
-P 5900 6650
-F 0 "S804" V 5980 6650 40  0000 L CNN
-F 1 "MH" H 5900 6705 30  0001 C CNN
-F 2 "TinyTiM_Libs:Screw_NPTH" H 5900 6805 30  0001 C CNN
-F 3 "" H 5900 6650 60  0001 C CNN
-	1    5900 6650
-	0    -1   -1   0
-$EndComp
 Text HLabel 950  2850 0    60   Input ~ 12
 5V
-Wire Wire Line
-	5100 6500 5100 6400
-Wire Wire Line
-	5100 6400 5400 6400
-Wire Wire Line
-	5400 6800 5400 6925
-Wire Wire Line
-	5400 6925 5100 6925
-Text Label 5100 6925 0    60   ~ 0
-GND
-Text Label 5400 6400 2    60   ~ 0
-5V
-$Comp
-L CONN_1 S806
-U 1 1 55311D21
-P 4500 6650
-F 0 "S806" V 4580 6650 40  0000 L CNN
-F 1 "CO_H" H 4500 6705 30  0001 C CNN
-F 2 "TinyTiM_Libs:Contact_SMD" H 4500 6805 30  0001 C CNN
-F 3 "" H 4500 6650 60  0001 C CNN
-	1    4500 6650
-	0    -1   -1   0
-$EndComp
-$Comp
-L CONN_1 S805
-U 1 1 55311DB5
-P 4100 6650
-F 0 "S805" V 4180 6650 40  0000 L CNN
-F 1 "DO_H" H 4100 6705 30  0001 C CNN
-F 2 "TinyTiM_Libs:Contact_SMD" H 4100 6805 30  0001 C CNN
-F 3 "" H 4100 6650 60  0001 C CNN
-	1    4100 6650
-	0    -1   -1   0
-$EndComp
-Wire Wire Line
-	4500 6800 4500 6925
-Wire Wire Line
-	4500 6925 4200 6925
-Wire Wire Line
-	4100 6800 4100 6925
-Wire Wire Line
-	4100 6925 3800 6925
-Text Label 3800 6925 0    60   ~ 0
-DO_H
-Text Label 4200 6925 0    60   ~ 0
-CO_H
 $Comp
 L APA102 U802

Commit message: layout complete. Gerbers pending
Parts:
- C3: renamed from C801; manf# (none) -> Value
- C4: renamed from C817; manf# (none) -> Value
- renumbered U801 to U57, U802 to U58, U803 to U59, U804 to U60, U805 to U61, U806 to U62, U807 to U63, U808 to U64
Changed lines of the file:
@@
 GND
 $Comp
-L APA102 U801
+L APA102 U57
 U 1 1 5118ABBB
 P 1700 1600
-F 0 "U801" H 1700 1900 40  0000 C CNB
+F 0 "U57" H 1700 1900 40  0000 C CNB
 F 1 "APA102" H 1700 1275 40  0000 C CNN
 F 2 "TinyTiM_Libs:APA102" H 1600 2000 60  0001 C CNN
@@
 CO_H
 $Comp
-L C2 C801
+L C2 C3
 U 1 1 51168961
 P 1800 2600
-F 0 "C801" H 1825 2700 50  0000 L CNN
+F 0 "C3" H 1825 2700 50  0000 L CNN
 F 1 "100n" H 1825 2500 50  0000 L CNN
 F 2 "TinyTiM_Libs:c_0805" H 1800 2600 50  0001 C CNN
 F 3 "" H 1800 2600 60  0001 C CNN
-F 4 "CAP CER 0.1UF 25V 10% X7R 0805" H 1800 2800 60  0001 L CNN "Field4"
-F 5 "100nF, 25V" H 1800 2900 60  0001 L CNN "Field5"
-F 6 "Surface Mount, MLCC" H 1800 3000 60  0001 L CNN "Field6"
-F 7 "Kemet" H 1800 3100 60  0001 L CNN "Field7"
-F 8 "C0805C104K3RACTU" H 1800 3200 60  0001 L CNN "Field8"
-F 9 "Digikey" H 1800 3300 60  0001 L CNN "Field9"
-F 10 "399-1168-1-ND" H 1800 3400 60  0001 L CNN "Field10"
-F 11 "http://www.digikey.com/product-detail/en/C0805C104K3RACTU/399-1168-1-ND/411443" H 1800 3500 60  0001 L CNN "Field11"
+F 4 "Value" H 1800 2600 60  0001 C CNN "manf#"
+F 5 "CAP CER 0.1UF 25V 10% X7R 0805" H 1800 2800 60  0001 L CNN "Field4"
+F 6 "100nF, 25V" H 1800 2900 60  0001 L CNN "Field5"
+F 7 "Surface Mount, MLCC" H 1800 3000 60  0001 L CNN "Field6"
+F 8 "Kemet" H 1800 3100 60  0001 L CNN "Field7"
+F 9 "C0805C104K3RACTU" H 1800 3200 60  0001 L CNN "Field8"
+F 10 "Digikey" H 1800 3300 60  0001 L CNN "Field9"
+F 11 "399-1168-1-ND" H 1800 3400 60  0001 L CNN "Field10"
+F 12 "http://www.digikey.com/product-detail/en/C0805C104K3RACTU/399-1168-1-ND/411443" H 1800 3500 60  0001 L CNN "Field11"
 	1    1800 2600
 	1    0    0    -1
@@
 GND
 $Comp
-L C_POL_1 C817
+L C_POL_1 C4
 U 1 1 5118AB61
 P 1250 6750
-F 0 "C817" H 1375 6725 50  0000 L CNN
+F 0 "C4" H 1375 6725 50  0000 L CNN
 F 1 "47u,8V" H 1375 6625 50  0000 L CNN
 F 2 "TinyTiM_Libs:c_2917" H 1250 6700 50  0001 C CNN
 F 3 "" H 1250 6750 60  0001 C CNN
-F 4 "CAP ALUM 47UF 8V 20% SMD" H 1250 6950 60  0001 L CNN "Field4"
-F 5 "47u,8V" H 1250 7050 60  0001 L CNN "Field5"
-F 6 "2917 (7343 Metric)" H 1250 7150 60  0001 L CNN "Field6"
-F 7 "Panasonic Electronic Components" H 1250 7250 60  0001 L CNN "Field7"
-F 8 "EEF-CD0K470R" H 1250 7350 60  0001 L CNN "Field8"
-F 9 "Digikey" H 1250 7450 60  0001 L CNN "Field9"
-F 10 "PCE3606CT-ND" H 1250 7550 60  0001 L CNN "Field10"
-F 11 "http://www.digikey.com/product-detail/en/EEF-CD0K470R/PCE3606CT-ND/614442" H 1250 7650 60  0001 L CNN "Field11"
+F 4 "Value" H 1250 6750 60  0001 C CNN "manf#"
+F 5 "CAP ALUM 47UF 8V 20% SMD" H 1250 6950 60  0001 L CNN "Field4"
+F 6 "47u,8V" H 1250 7050 60  0001 L CNN "Field5"
+F 7 "2917 (7343 Metric)" H 1250 7150 60  0001 L CNN "Field6"
+F 8 "Panasonic Electronic Components" H 1250 7250 60  0001 L CNN "Field7"
+F 9 "EEF-CD0K470R" H 1250 7350 60  0001 L CNN "Field8"
+F 10 "Digikey" H 1250 7450 60  0001 L CNN "Field9"
+F 11 "PCE3606CT-ND" H 1250 7550 60  0001 L CNN "Field10"
+F 12 "http://www.digikey.com/product-detail/en/EEF-CD0K470R/PCE3606CT-ND/614442" H 1250 7650 60  0001 L CNN "Field11"
 	1    1250 6750
 	1    0    0    -1
@@
 5V
 $Comp
-L APA102 U802
+L APA102 U58
 U 1 1 56C06E0E
 P 2900 1600
-F 0 "U802" H 2900 1900 40  0000 C CNB
+F 0 "U58" H 2900 1900 40  0000 C CNB
 F 1 "APA102" H 2900 1275 40  0000 C CNN
 F 2 "TinyTiM_Libs:APA102" H 2800 2000 60  0001 C CNN
@@
 $EndComp
 $Comp
-L APA102 U803
+L APA102 U59
 U 1 1 56C06E52
 P 4100 1600
-F 0 "U803" H 4100 1900 40  0000 C CNB
+F 0 "U59" H 4100 1900 40  0000 C CNB
 F 1 "APA102" H 4100 1275 40  0000 C CNN
 F 2 "TinyTiM_Libs:APA102" H 4000 2000 60  0001 C CNN
@@
 $EndComp
 $Comp
-L APA102 U804
+L APA102 U60
 U 1 1 56C06F1D
 P 5300 1600
-F 0 "U804" H 5300 1900 40  0000 C CNB
+F 0 "U60" H 5300 1900 40  0000 C CNB
 F 1 "APA102" H 5300 1275 40  0000 C CNN
 F 2 "TinyTiM_Libs:APA102" H 5200 2000 60  0001 C CNN
@@
 $EndComp
 $Comp
-L APA102 U805
+L APA102 U61
 U 1 1 56C06FBB
 P 6500 1600
-F 0 "U805" H 6500 1900 40  0000 C CNB
+F 0 "U61" H 6500 1900 40  0000 C CNB
 F 1 "APA102" H 6500 1275 40  0000 C CNN
 F 2 "TinyTiM_Libs:APA102" H 6400 2000 60  0001 C CNN
@@
 $EndComp
 $Comp
-L APA102 U806
+L APA102 U62
 U 1 1 56C07772
 P 7700 1600
-F 0 "U806" H 7700 1900 40  0000 C CNB
+F 0 "U62" H 7700 1900 40  0000 C CNB
 F 1 "APA102" H 7700 1275 40  0000 C CNN
 F 2 "TinyTiM_Libs:APA102" H 7600 2000 60  0001 C CNN
@@
 $EndComp
 $Comp
-L APA102 U807
+L APA102 U63
 U 1 1 56C077C2
 P 8900 1600
-F 0 "U807" H 8900 1900 40  0000 C CNB
+F 0 "U63" H 8900 1900 40  0000 C CNB
 F 1 "APA102" H 8900 1275 40  0000 C CNN
 F 2 "TinyTiM_Libs:APA102" H 8800 2000 60  0001 C CNN
@@
 $EndComp
 $Comp
-L APA102 U808
+L APA102 U64
 U 1 1 56C07914
 P 10100 1600
-F 0 "U808" H 10100 1900 40  0000 C CNB
+F 0 "U64" H 10100 1900 40  0000 C CNB
 F 1 "APA102" H 10100 1275 40  0000 C CNN
 F 2 "TinyTiM_Libs:APA102" H 10000 2000 60  0001 C CNN
